File: Control de Gabinetes/esp32.sch (KiCad schematic (older format))
At the start: 0 parts

Commit message: Avance 1/07/2021
Parts:
- added C?: 0.1uf, Capacitor_SMD:C_0805_2012Metric, symbol Device:C
- added C?: 10uf, Capacitor_SMD:C_0805_2012Metric, symbol Device:C
- added J?: Conn_01x04, symbol Connector_Generic:Conn_01x04
- added R? (x3): 10K, Resistor_SMD:R_0805_2012Metric, symbol Device:R
- added SW?: SW_Push, Button_Switch_SMD:SW_SPST_TL3342, symbol Switch:SW_Push
- added U1: ESP32-WROOM-32D, RF_Module:ESP32-WROOM-32, symbol RF_Module:ESP32-WROOM-32D
Connections:
- new net +3V3: C?.1, C?.2, R?.1, R?.1, R?.2, U1.2 (VDD)
- new net GND: C?.1, C?.2, J?.4 (Pin_4), SW?.1, U1.1 (GND), U1.15 (GND), U1.38 (GND), U1.39 (GND)
- new net RESET: J?.3 (Pin_3), R?.1, SW?.2, U1.3 (EN)
- new net RX: J?.2 (Pin_2), U1.34 (RXD0/IO3)
- new net SCL: R?.2, U1.8 (IO32)
- new net SDA: R?.2, U1.9 (IO33)
- new net TX: J?.1 (Pin_1), U1.35 (TXD0/IO1)
Other:
- note added: "Cual es el valor de la bobina que\n debo colocar de desacoplamiento?\nAparte del VCC y GND del micro donde\nmas se debe colocar desacoplamiento?\n"
