File: Control de Gabinetes/esp32.sch (KiCad schematic (older format))
At the start: 8 parts, among them U1 ESP32-WROOM-32D

Commit message: avance 6/07
Parts:
- added L?: 330 ohm, symbol Device:L
- J?: footprint (none) -> Connector_Molex:Molex_KK-254_AE-6410-04A_1x04_P2.54mm_Vertical
Connections:
- net labels added: S_APERTURA, S_HUMEDAD, S_MOVIMIENTO
- wire segments 41 -> 51
Other:
- moved on the sheet: J?, R?, SW?
Changed lines of the file:
@@
 $Descr A4 11693 8268
 encoding utf-8
-Sheet 2 6
+Sheet 6 6
 Title ""
 Date ""
@@
 L power:+3.3V #PWR?
 U 1 1 60DD778F
-P 5650 1700
-F 0 "#PWR?" H 5650 1550 50  0001 C CNN
-F 1 "+3.3V" H 5665 1873 50  0000 C CNN
-F 2 "" H 5650 1700 50  0001 C CNN
-F 3 "" H 5650 1700 50  0001 C CNN
-	1    5650 1700
+P 5650 1200
+F 0 "#PWR?" H 5650 1050 50  0001 C CNN
+F 1 "+3.3V" H 5665 1373 50  0000 C CNN
+F 2 "" H 5650 1200 50  0001 C CNN
+F 3 "" H 5650 1200 50  0001 C CNN
+	1    5650 1200
 	1    0    0    -1
 $EndComp
@@
 L Device:R R?
 U 1 1 60DDAD0C
-P 9100 3500
-F 0 "R?" V 8893 3500 50  0000 C CNN
-F 1 "10K" H 8984 3500 50  0000 C CNN
-F 2 "Resistor_SMD:R_0805_2012Metric" V 9030 3500 50  0001 C CNN
-F 3 "~" H 9100 3500 50  0001 C CNN
-	1    9100 3500
+P 9250 3100
+F 0 "R?" V 9043 3100 50  0000 C CNN
+F 1 "10K" H 9134 3100 50  0000 C CNN
+F 2 "Resistor_SMD:R_0805_2012Metric" V 9180 3100 50  0001 C CNN
+F 3 "~" H 9250 3100 50  0001 C CNN
+	1    9250 3100
 	0    1    1    0
 $EndComp
@@
 L Switch:SW_Push SW?
 U 1 1 60DE8A30
-P 9100 3700
-F 0 "SW?" H 9100 3650 50  0000 C CNN
-F 1 "SW_Push" H 9100 3550 50  0000 C CNN
-F 2 "Button_Switch_SMD:SW_SPST_TL3342" H 9100 3893 50  0001 C CNN
-F 3 "~" H 9100 3900 50  0001 C CNN
-	1    9100 3700
+P 9250 3300
+F 0 "SW?" H 9250 3250 50  0000 C CNN
+F 1 "SW_Push" H 9250 3150 50  0000 C CNN
+F 2 "Button_Switch_SMD:SW_SPST_TL3342" H 9250 3493 50  0001 C CNN
+F 3 "~" H 9250 3500 50  0001 C CNN
+	1    9250 3300
 	1    0    0    -1
 $EndComp
@@
 L power:GND #PWR?
 U 1 1 60DEAE68
-P 8750 3900
-F 0 "#PWR?" H 8750 3650 50  0001 C CNN
-F 1 "GND" H 8755 3727 50  0000 C CNN
-F 2 "" H 8750 3900 50  0001 C CNN
-F 3 "" H 8750 3900 50  0001 C CNN
-	1    8750 3900
-	1    0    0    -1
-$EndComp
-Wire Wire Line
-	8750 3700 8750 3900
-Text Notes 5000 1450 0    50   ~ 0
+P 8900 3500
+F 0 "#PWR?" H 8900 3250 50  0001 C CNN
+F 1 "GND" H 8905 3327 50  0000 C CNN
+F 2 "" H 8900 3500 50  0001 C CNN
+F 3 "" H 8900 3500 50  0001 C CNN
+	1    8900 3500
+	1    0    0    -1
+$EndComp
+Wire Wire Line
+	8900 3300 8900 3500
+Text Notes 5000 900  0    50   ~ 0
 Cual es el valor de la bobina que\n debo colocar de desacoplamiento?\nAparte del VCC y GND del micro donde\nmas se debe colocar desacoplamiento?\n
 $Comp
@@
 L power:+3.3V #PWR?
 U 1 1 60DFF360
-P 8750 3250
-F 0 "#PWR?" H 8750 3100 50  0001 C CNN
-F 1 "+3.3V" H 8765 3423 50  0000 C CNN
-F 2 "" H 8750 3250 50  0001 C CNN
-F 3 "" H 8750 3250 50  0001 C CNN
-	1    8750 3250
-	1    0    0    -1
-$EndComp
-Wire Wire Line
-	8750 3250 8750 3500
+P 8900 2850
+F 0 "#PWR?" H 8900 2700 50  0001 C CNN
+F 1 "+3.3V" H 8915 3023 50  0000 C CNN
+F 2 "" H 8900 2850 50  0001 C CNN
+F 3 "" H 8900 2850 50  0001 C CNN
+	1    8900 2850
+	1    0    0    -1
+$EndComp
+Wire Wire Line
+	8900 2850 8900 3100
 $Comp
 L Connector_Generic:Conn_01x04 J?
 U 1 1 60E0C30F
-P 9400 2100
-F 0 "J?" H 9480 2092 50  0000 L CNN
-F 1 "Conn_01x04" H 9480 2001 50  0000 L CNN
-F 2 "" H 9400 2100 50  0001 C CNN
-F 3 "~" H 9400 2100 50  0001 C CNN
-	1    9400 2100
-	1    0    0    -1
-$EndComp
-Wire Wire Line
-	9200 2300 8950 2300
-Wire Wire Line
-	8950 2000 9200 2000
-Wire Wire Line
-	9200 2100 8950 2100
-Wire Wire Line
-	9200 2200 8950 2200
+P 9500 1900
+F 0 "J?" H 9580 1892 50  0000 L CNN
+F 1 "Conn_01x04" H 9580 1801 50  0000 L CNN
+F 2 "Connector_Molex:Molex_KK-254_AE-6410-04A_1x04_P2.54mm_Vertical" H 9500 1900 50  0001 C CNN
+F 3 "~" H 9500 1900 50  0001 C CNN
+	1    9500 1900
+	1    0    0    -1
+$EndComp
+Wire Wire Line
+	9300 2100 9050 2100
+Wire Wire Line
+	9050 1800 9300 1800
+Wire Wire Line
+	9300 1900 9050 1900
+Wire Wire Line
+	9300 2000 9050 2000
 Wire Wire Line
 	6250 2400 6450 2400
@@
 Text Label 6450 2400 0    50   ~ 0
 RX
-Text Label 8950 2000 2    50   ~ 0
+Text Label 9050 1800 2    50   ~ 0
 TX
-Text Label 8950 2100 2    50   ~ 0
+Text Label 9050 1900 2    50   ~ 0
 RX
-Text Label 8950 2200 2    50   ~ 0
+Text Label 9050 2000 2    50   ~ 0
 RESET
 $Comp
 L power:GND #PWR?
 U 1 1 60E12E44
-P 8950 2300
-F 0 "#PWR?" H 8950 2050 50  0001 C CNN
-F 1 "GND" V 8955 2172 50  0000 R CNN
-F 2 "" H 8950 2300 50  0001 C CNN
-F 3 "" H 8950 2300 50  0001 C CNN
-	1    8950 2300
+P 9050 2100
+F 0 "#PWR?" H 9050 1850 50  0001 C CNN
+F 1 "GND" V 9055 1972 50  0000 R CNN
+F 2 "" H 9050 2100 50  0001 C CNN
+F 3 "" H 9050 2100 50  0001 C CNN
+	1    9050 2100
 	0    1    1    0
 $EndComp
 Wire Wire Line
-	8950 3500 8750 3500
-Wire Wire Line
-	8900 3700 8750 3700
-Wire Wire Line
-	9300 3700 9450 3700
-Wire Wire Line
-	9450 3700 9450 3500
-Wire Wire Line
-	9450 3500 9250 3500
-Wire Wire Line
-	9650 3500 9450 3500
-Connection ~ 9450 3500
-Text Label 9650 3500 0    50   ~ 0
+	9100 3100 8900 3100
+Wire Wire Line
+	9050 3300 8900 3300
+Wire Wire Line
+	9450 3300 9600 3300
+Wire Wire Line
+	9600 3300 9600 3100
+Wire Wire Line
+	9600 3100 9400 3100
+Wire Wire Line
+	9800 3100 9600 3100
+Connection ~ 9600 3100
+Text Label 9800 3100 0    50   ~ 0
 RESET
 Wire Wire Line
@@
 L power:+3.3V #PWR?
 U 1 1 60E3AA57
-P 9450 4600
-F 0 "#PWR?" H 9450 4450 50  0001 C CNN
-F 1 "+3.3V" H 9465 4773 50  0000 C CNN
-F 2 "" H 9450 4600 50  0001 C CNN
-F 3 "" H 9450 4600 50  0001 C CNN
-	1    9450 4600
+P 9700 4850
+F 0 "#PWR?" H 9700 4700 50  0001 C CNN
+F 1 "+3.3V" H 9715 5023 50  0000 C CNN
+F 2 "" H 9700 4850 50  0001 C CNN
+F 3 "" H 9700 4850 50  0001 C CNN
+	1    9700 4850
 	1    0    0    -1
 $EndComp
@@
 L Device:R R?
 U 1 1 60E3B498
-P 9100 4800
-F 0 "R?" V 8893 4800 50  0000 C CNN
-F 1 "10K" V 8984 4800 50  0000 C CNN
-F 2 "Resistor_SMD:R_0805_2012Metric" V 9030 4800 50  0001 C CNN
-F 3 "~" H 9100 4800 50  0001 C CNN
-	1    9100 4800
+P 9350 5050
+F 0 "R?" V 9143 5050 50  0000 C CNN
+F 1 "10K" V 9234 5050 50  0000 C CNN
+F 2 "Resistor_SMD:R_0805_2012Metric" V 9280 5050 50  0001 C CNN
+F 3 "~" H 9350 5050 50  0001 C CNN
+	1    9350 5050
 	0    1    1    0
 $EndComp
@@
 L Device:R R?
 U 1 1 60E3CE15
-P 9100 5100
-F 0 "R?" V 8893 5100 50  0000 C CNN
-F 1 "10K" V 8984 5100 50  0000 C CNN
-F 2 "Resistor_SMD:R_0805_2012Metric" V 9030 5100 50  0001 C CNN
-F 3 "~" H 9100 5100 50  0001 C CNN
-	1    9100 5100
+P 9350 5350
+F 0 "R?" V 9143 5350 50  0000 C CNN
+F 1 "10K" V 9234 5350 50  0000 C CNN
+F 2 "Resistor_SMD:R_0805_2012Metric" V 9280 5350 50  0001 C CNN
+F 3 "~" H 9350 5350 50  0001 C CNN
+	1    9350 5350
 	0    1    1    0
 $EndComp
 Wire Wire Line
-	9450 4800 9450 4600
-Wire Wire Line
-	9250 4800 9450 4800
-Wire Wire Line
-	9250 5100 9450 5100
-Wire Wire Line
-	9450 5100 9450 4800
-Connection ~ 9450 4800
-Wire Wire Line
-	8750 4800 8950 4800
-Wire Wire Line
-	8750 5100 8950 5100
-Text Label 8750 4800 2    50   ~ 0
+	9700 5050 9700 4850
+Wire Wire Line
+	9500 5050 9700 5050
+Wire Wire Line
+	9500 5350 9700 5350
+Wire Wire Line
+	9700 5350 9700 5050
+Connection ~ 9700 5050
+Wire Wire Line
+	9000 5050 9050 5050
+Wire Wire Line
+	9000 5350 9050 5350
+Text Label 9000 5050 2    50   ~ 0
 SDA
-Text Label 8750 5100 2    50   ~ 0
+Text Label 9000 5350 2    50   ~ 0
 SCL
-Wire Wire Line
-	6450 4100 6250 4100
-Wire Wire Line
-	6450 4200 6250 4200
-Text Label 6450 4200 0    50   ~ 0
+Text Label 6450 3500 0    50   ~ 0
 SDA
-Text Label 6450 4100 0    50   ~ 0
+Text Label 6450 3600 0    50   ~ 0
 SCL
+$Comp
+L Device:L L?
+U 1 1 60E365EB
+P 5650 1550
+F 0 "L?" H 5702 1596 50  0000 L CNN
+F 1 "330 ohm" H 5702 1505 50  0000 L CNN
+F 2 "" H 5650 1550 50  0001 C CNN
+F 3 "~" H 5650 1550 50  0001 C CNN
+	1    5650 1550
+	1    0    0    -1
+$EndComp
+Wire Wire Line
+	5650 1200 5650 1400
+Wire Wire Line
+	9000 4950 9050 4950
+Wire Wire Line
+	9050 4950 9050 5050
+Connection ~ 9050 5050
+Wire Wire Line
+	9050 5050 9200 5050
+Wire Wire Line
+	9000 5250 9050 5250
+Wire Wire Line
+	9050 5250 9050 5350
+Connection ~ 9050 5350
+Wire Wire Line
+	9050 5350 9200 5350
+Text HLabel 9000 4950 0    50   BiDi ~ 0
+SDA
+Text HLabel 9000 5250 0    50   BiDi ~ 0
+SCL
+Wire Wire Line
+	6450 3500 6250 3500
+Wire Wire Line
+	6450 3600 6250 3600
+Wire Wire Line
+	6450 2900 6250 2900
+Wire Wire Line
+	6450 2700 6250 2700
+Wire Wire Line
+	6450 2800 6250 2800
+Text HLabel 6450 2700 2    50   Input ~ 0
+S_HUMEDAD
+Text HLabel 6450 2800 2    50   Input ~ 0
+S_MOVIMIENTO
+Text HLabel 6450 2900 2    50   Input ~ 0
+S_APERTURA
 $EndSCHEMATC

Commit message: AVANCE 7/7/2021
Parts:
- removed L?: 330 ohm, symbol Device:L
Connections:
- net labels added: CS, DIO0, MISO, MOSI, PWRKEY, RESET_L, RX2, SCK, SLEEP1, TX2
- wire segments 51 -> 60
Other:
- note removed: "Cual es el valor de la bobina que\n debo colocar de desacoplamiento?\nAparte del VCC y GND del micro donde\nmas se debe colocar desacoplamiento?\n"
Changed lines of the file:
@@
 $Descr A4 11693 8268
 encoding utf-8
-Sheet 6 6
+Sheet 5 6
 Title ""
 Date ""
@@
 L power:+3.3V #PWR?
 U 1 1 60DD778F
-P 5650 1200
-F 0 "#PWR?" H 5650 1050 50  0001 C CNN
-F 1 "+3.3V" H 5665 1373 50  0000 C CNN
-F 2 "" H 5650 1200 50  0001 C CNN
-F 3 "" H 5650 1200 50  0001 C CNN
-	1    5650 1200
-	1    0    0    -1
-$EndComp
-Wire Wire Line
-	5650 1700 5650 1900
+P 5650 1700
+F 0 "#PWR?" H 5650 1550 50  0001 C CNN
+F 1 "+3.3V" H 5665 1873 50  0000 C CNN
+F 2 "" H 5650 1700 50  0001 C CNN
+F 3 "" H 5650 1700 50  0001 C CNN
+	1    5650 1700
+	1    0    0    -1
+$EndComp
 $Comp
 L power:GND #PWR?
@@
 Wire Wire Line
 	8900 3300 8900 3500
-Text Notes 5000 900  0    50   ~ 0
-Cual es el valor de la bobina que\n debo colocar de desacoplamiento?\nAparte del VCC y GND del micro donde\nmas se debe colocar desacoplamiento?\n
 $Comp
 L power:GND #PWR?
@@
 Text Label 6450 3600 0    50   ~ 0
 SCL
-$Comp
-L Device:L L?
-U 1 1 60E365EB
-P 5650 1550
-F 0 "L?" H 5702 1596 50  0000 L CNN
-F 1 "330 ohm" H 5702 1505 50  0000 L CNN
-F 2 "" H 5650 1550 50  0001 C CNN
-F 3 "~" H 5650 1550 50  0001 C CNN
-	1    5650 1550
-	1    0    0    -1
-$EndComp
-Wire Wire Line
-	5650 1200 5650 1400
 Wire Wire Line
 	9000 4950 9050 4950
@@
 Text HLabel 6450 2900 2    50   Input ~ 0
 S_APERTURA
+Wire Wire Line
+	5650 1900 5650 1700
+Wire Wire Line
+	6450 3200 6250 3200
+Wire Wire Line
+	6450 3100 6250 3100
+Text HLabel 6450 3100 2    50   Input ~ 0
+RX2
+Text HLabel 6450 3200 2    50   Output ~ 0
+TX2
+Wire Wire Line
+	6450 3000 6250 3000
+Text HLabel 6450 3000 2    50   Output ~ 0
+PWRKEY
+Wire Wire Line
+	6450 3800 6250 3800
+Text HLabel 6450 3800 2    50   Output ~ 0
+SLEEP1
+Wire Wire Line
+	6450 3900 6250 3900
+Text HLabel 6450 3900 2    50   Output ~ 0
+RESET_L
+Wire Wire Line
+	6450 3300 6250 3300
+Text HLabel 6450 3300 2    50   BiDi ~ 0
+SCK
+Wire Wire Line
+	6450 3400 6250 3400
+Text HLabel 6450 3400 2    50   Input ~ 0
+MISO
+Wire Wire Line
+	6450 3700 6250 3700
+Text HLabel 6450 3700 2    50   Output ~ 0
+MOSI
+Wire Wire Line
+	6450 2300 6250 2300
+Text HLabel 6450 2300 2    50   Output ~ 0
+CS
+Wire Wire Line
+	6450 4000 6250 4000
+Text HLabel 6450 4000 2    50   Output ~ 0
+DIO0
 $EndSCHEMATC

Commit message: AVANCE 13/07/2021
Parts:
- gave numbers to parts that had none: 7
Connections:
- net CS: now also U1.29 (IO5); no longer U1.24 (IO2)
- net TX_SWITCH: now reaches U1.8 (IO32)
- net RX_SWITCH: now reaches U1.9 (IO33)
Other:
- note added: "SOLO________>\nENTRADAS"
Changed lines of the file:
@@
 $EndComp
 $Comp
-L Device:C C?
+L Device:C C6
 U 1 1 60AF11EF
 P 1800 1850
-F 0 "C?" H 1915 1896 50  0000 L CNN
+F 0 "C6" H 1915 1896 50  0000 L CNN
 F 1 "0.1uf" H 1915 1805 50  0000 L CNN
 F 2 "Capacitor_SMD:C_0805_2012Metric" H 1838 1700 50  0001 C CNN
@@
 $EndComp
 $Comp
-L Device:C C?
+L Device:C C5
 U 1 1 60AF1541
 P 1400 1850
-F 0 "C?" H 1285 1804 50  0000 R CNN
+F 0 "C5" H 1285 1804 50  0000 R CNN
 F 1 "10uf" H 1285 1895 50  0000 R CNN
 F 2 "Capacitor_SMD:C_0805_2012Metric" H 1438 1700 50  0001 C CNN
@@
 	1800 2250 1800 2000
 $Comp
-L power:+3.3V #PWR?
+L power:+3.3V #PWR0132
 U 1 1 60DD778F
 P 5650 1700
-F 0 "#PWR?" H 5650 1550 50  0001 C CNN
+F 0 "#PWR0132" H 5650 1550 50  0001 C CNN
 F 1 "+3.3V" H 5665 1873 50  0000 C CNN
 F 2 "" H 5650 1700 50  0001 C CNN
@@
 $EndComp
 $Comp
-L power:GND #PWR?
+L power:GND #PWR0133
 U 1 1 60DD8C2E
 P 5650 4900
-F 0 "#PWR?" H 5650 4650 50  0001 C CNN
+F 0 "#PWR0133" H 5650 4650 50  0001 C CNN
 F 1 "GND" H 5655 4727 50  0000 C CNN
 F 2 "" H 5650 4900 50  0001 C CNN
@@
 	5650 4700 5650 4900
 $Comp
-L Device:R R?
+L Device:R R10
 U 1 1 60DDAD0C
 P 9250 3100
-F 0 "R?" V 9043 3100 50  0000 C CNN
+F 0 "R10" V 9043 3100 50  0000 C CNN
 F 1 "10K" H 9134 3100 50  0000 C CNN
 F 2 "Resistor_SMD:R_0805_2012Metric" V 9180 3100 50  0001 C CNN
@@
 $EndComp
 $Comp
-L Switch:SW_Push SW?
+L Switch:SW_Push SW1
 U 1 1 60DE8A30
 P 9250 3300
-F 0 "SW?" H 9250 3250 50  0000 C CNN
+F 0 "SW1" H 9250 3250 50  0000 C CNN
 F 1 "SW_Push" H 9250 3150 50  0000 C CNN
 F 2 "Button_Switch_SMD:SW_SPST_TL3342" H 9250 3493 50  0001 C CNN
@@
 $EndComp
 $Comp
-L power:GND #PWR?
+L power:GND #PWR0134
 U 1 1 60DEAE68
 P 8900 3500
-F 0 "#PWR?" H 8900 3250 50  0001 C CNN
+F 0 "#PWR0134" H 8900 3250 50  0001 C CNN
 F 1 "GND" H 8905 3327 50  0000 C CNN
 F 2 "" H 8900 3500 50  0001 C CNN
@@
 	8900 3300 8900 3500
 $Comp
-L power:GND #PWR?
+L power:GND #PWR0135
 U 1 1 60DF3D45
 P 1600 2450
-F 0 "#PWR?" H 1600 2200 50  0001 C CNN
+F 0 "#PWR0135" H 1600 2200 50  0001 C CNN
 F 1 "GND" H 1605 2277 50  0000 C CNN
 F 2 "" H 1600 2450 50  0001 C CNN
@@
 $EndComp
 $Comp
-L power:+3.3V #PWR?
+L power:+3.3V #PWR0136
 U 1 1 60DF56E9
 P 1600 1300
-F 0 "#PWR?" H 1600 1150 50  0001 C CNN
+F 0 "#PWR0136" H 1600 1150 50  0001 C CNN
 F 1 "+3.3V" H 1615 1473 50  0000 C CNN
 F 2 "" H 1600 1300 50  0001 C CNN
@@
 	1600 2350 1600 2250
 $Comp
-L power:+3.3V #PWR?
+L power:+3.3V #PWR0137
 U 1 1 60DFF360
 P 8900 2850
-F 0 "#PWR?" H 8900 2700 50  0001 C CNN
+F 0 "#PWR0137" H 8900 2700 50  0001 C CNN
 F 1 "+3.3V" H 8915 3023 50  0000 C CNN
 F 2 "" H 8900 2850 50  0001 C CNN
@@
 	8900 2850 8900 3100
 $Comp
-L Connector_Generic:Conn_01x04 J?
+L Connector_Generic:Conn_01x04 J6
 U 1 1 60E0C30F
 P 9500 1900
-F 0 "J?" H 9580 1892 50  0000 L CNN
+F 0 "J6" H 9580 1892 50  0000 L CNN
 F 1 "Conn_01x04" H 9580 1801 50  0000 L CNN
 F 2 "Connector_Molex:Molex_KK-254_AE-6410-04A_1x04_P2.54mm_Vertical" H 9500 1900 50  0001 C CNN
@@
 RESET
 $Comp
-L power:GND #PWR?
+L power:GND #PWR0138
 U 1 1 60E12E44
 P 9050 2100
-F 0 "#PWR?" H 9050 1850 50  0001 C CNN
+F 0 "#PWR0138" H 9050 1850 50  0001 C CNN
 F 1 "GND" V 9055 1972 50  0000 R CNN
 F 2 "" H 9050 2100 50  0001 C CNN
@@
 RESET
 $Comp
-L power:+3.3V #PWR?
+L power:+3.3V #PWR0139
 U 1 1 60E3AA57
 P 9700 4850
-F 0 "#PWR?" H 9700 4700 50  0001 C CNN
+F 0 "#PWR0139" H 9700 4700 50  0001 C CNN
 F 1 "+3.3V" H 9715 5023 50  0000 C CNN
 F 2 "" H 9700 4850 50  0001 C CNN
@@
 $EndComp
 $Comp
-L Device:R R?
+L Device:R R11
 U 1 1 60E3B498
 P 9350 5050
-F 0 "R?" V 9143 5050 50  0000 C CNN
+F 0 "R11" V 9143 5050 50  0000 C CNN
 F 1 "10K" V 9234 5050 50  0000 C CNN
 F 2 "Resistor_SMD:R_0805_2012Metric" V 9280 5050 50  0001 C CNN
@@
 $EndComp
 $Comp
-L Device:R R?
+L Device:R R12
 U 1 1 60E3CE15
 P 9350 5350
-F 0 "R?" V 9143 5350 50  0000 C CNN
+F 0 "R12" V 9143 5350 50  0000 C CNN
 F 1 "10K" V 9234 5350 50  0000 C CNN
 F 2 "Resistor_SMD:R_0805_2012Metric" V 9280 5350 50  0001 C CNN
@@
 MOSI
 Wire Wire Line
-	6450 2300 6250 2300
-Text HLabel 6450 2300 2    50   Output ~ 0
+	6450 2600 6250 2600
+Text HLabel 6450 2600 2    50   Output ~ 0
 CS
 Wire Wire Line
@@
 Text HLabel 6450 4000 2    50   Output ~ 0
 DIO0
+Wire Wire Line
+	6450 4100 6250 4100
+Wire Wire Line
+	6450 4200 6250 4200
+Text HLabel 6450 4100 2    50   Output ~ 0
+TX_SWITCH
+Text HLabel 6450 4200 2    50   Output ~ 0
+RX_SWITCH
+Text Notes 4500 2400 0    39   ~ 0
+SOLO________>\nENTRADAS
 $EndSCHEMATC

Commit message: avance 19/07
Parts:
- added J11, J12, J13: Conn_01x02_Male, Connector_PinHeader_2.54mm:PinHeader_1x02_P2.54mm_Vertical, symbol Connector:Conn_01x02_Male
- added Q6, Q7, Q8: PN2222A, Package_TO_SOT_THT:TO-92_Inline, symbol Transistor_BJT:PN2222A
- added R29, R30, R31: R, Resistor_SMD:R_0805_2012Metric, symbol Device:R
- added R32: 10K, Resistor_SMD:R_0805_2012Metric, symbol Device:R
- added SW2: ARRANQUE, Button_Switch_SMD:SW_SPST_TL3342, symbol Switch:SW_Push
- J6: footprint Connector_Molex:Molex_KK-254_AE-6410-04A_1x04_P2.54mm_Vertical -> Connector_Molex:Molex_KK-254_AE-6410-05A_1x05_P2.54mm_Vertical; symbol Connector_Generic:Conn_01x04 -> Connector_Generic:Conn_01x05
- SW1: value SW_Push -> RESET
Connections:
- net +3V3: now also R32.2
- net GND: now also J6.5 (Pin_5), SW2.1; no longer J6.4 (Pin_4)
- net RESET: now also Q6.1 (E), R30.2, R31.2; no longer R10.1, SW1.2, U1.3 (EN)
- net RELAY3: now reaches U1.17 (SHD/SD2)
- net RELAY4: now reaches U1.18 (SWP/SD3)
- net IO2: now reaches U1.24 (IO2)
- net IO2: now also J13.2 (Pin_2)
- net IO0: now reaches U1.25 (IO0)
- net IO0: now also J12.2 (Pin_2), R32.1, SW2.2
- net RELAY1: now reaches U1.6 (IO34)
- net RELAY2: now reaches U1.7 (IO35)
- new net: Q6.2 (B), R29.1
- new net: J11.1 (Pin_1), Q6.3 (C)
- new net: J12.1 (Pin_1), Q7.1 (E)
- new net: Q7.2 (B), R30.1
- new net: J13.1 (Pin_1), Q8.1 (E)
- new net: Q8.2 (B), R31.1
- new net DTR: J6.4 (Pin_4), Q7.3 (C), Q8.3 (C), R29.2
- new net EN: J11.2 (Pin_2), R10.1, SW1.2, U1.3 (EN)
Other:
- note added: "AUTO PROGRAMACION"
- moved on the sheet: C5, C6, R11, R12

Commit message: avance2 19/07/2021
Parts:
- Q6, Q7, Q8: footprint Package_TO_SOT_THT:TO-92_Inline -> Package_TO_SOT_SMD:SOT-23
- R29, R30, R31: value R -> 10K
- U1: footprint RF_Module:ESP32-WROOM-32 -> RF_Module:ESP32-WROOM-32U
Connections:
- net RX_SWITCH is gone; now on net RELAY4: U1.9 (IO33)
- net TX_SWITCH is gone; now on net RELAY3: U1.8 (IO32)
- net RELAY3: no longer U1.17 (SHD/SD2)
- net RELAY4: no longer U1.18 (SWP/SD3)
- net S_HUMEDAD: now also U1.16 (IO13); no longer U1.14 (IO12)
- net S_MOVIMIENTO: now also U1.14 (IO12); no longer U1.16 (IO13)

Commit message: avance 20/07/2021
Parts:
- removed R10, R32: 10K, Resistor_SMD:R_0805_2012Metric, symbol Device:R
- added C7, C8: 0.1uf, Capacitor_SMD:C_0805_2012Metric, symbol Device:C
Connections:
- net DIO0: now also U1.13 (IO14); no longer U1.12 (IO27)
- net EN: now also C7.2
- net GND: now also C7.1, C8.2
- net IO0: now also C8.1
- net PWRKEY: now also U1.16 (IO13); no longer U1.23 (IO15)
- net RESET_L: now also U1.14 (IO12); no longer U1.11 (IO26)
- net SLEEP1: now also U1.23 (IO15); no longer U1.10 (IO25)
- net S_APERTURA: now also U1.12 (IO27); no longer U1.13 (IO14)
- net S_HUMEDAD: now also U1.11 (IO26); no longer U1.16 (IO13)
- net S_MOVIMIENTO: now also U1.10 (IO25); no longer U1.14 (IO12)
Changed lines of the file:
@@
 Wire Wire Line
 	6450 4200 6250 4200
-Text HLabel 6450 4000 2    50   Output ~ 0
+Text HLabel 6450 2900 2    50   Output ~ 0
 DIO0
 Wire Wire Line
 	6450 4000 6250 4000
-Text HLabel 6450 3900 2    50   Output ~ 0
+Text HLabel 6450 2700 2    50   Output ~ 0
 RESET_L
 Wire Wire Line
 	6450 3900 6250 3900
-Text HLabel 6450 3800 2    50   Output ~ 0
+Text HLabel 6450 3000 2    50   Output ~ 0
 SLEEP1
 Wire Wire Line
@@
 Wire Wire Line
 	6450 3300 6250 3300
-Text HLabel 6450 3000 2    50   Output ~ 0
+Text HLabel 6450 2800 2    50   Output ~ 0
 PWRKEY
 Wire Wire Line
 	6450 3000 6250 3000
-Text HLabel 6450 2900 2    50   Input ~ 0
+Text HLabel 6450 4000 2    50   Input ~ 0
 S_APERTURA
 Wire Wire Line
 	6450 2900 6250 2900
-Text HLabel 6450 2700 2    50   Input ~ 0
+Text HLabel 6450 3800 2    50   Input ~ 0
 S_MOVIMIENTO
 Wire Wire Line
 	6450 2800 6250 2800
-Text HLabel 6450 2800 2    50   Input ~ 0
+Text HLabel 6450 3900 2    50   Input ~ 0
 S_HUMEDAD
 Wire Wire Line
@@
 Text Label 9800 4350 0    50   ~ 0
 IO0
-Connection ~ 9600 4350
 Wire Wire Line
 	9800 4350 9600 4350
 Wire Wire Line
-	9600 4350 9400 4350
-Wire Wire Line
 	9600 4550 9600 4350
 Wire Wire Line
@@
 Wire Wire Line
 	9050 4550 8900 4550
-Wire Wire Line
-	9100 4350 8900 4350
-Wire Wire Line
-	8900 4100 8900 4350
-$Comp
-L power:+3.3V #PWR0145
-U 1 1 60F0477E
-P 8900 4100
-F 0 "#PWR0145" H 8900 3950 50  0001 C CNN
-F 1 "+3.3V" H 8915 4273 50  0000 C CNN
-F 2 "" H 8900 4100 50  0001 C CNN
-F 3 "" H 8900 4100 50  0001 C CNN
-	1    8900 4100
-	1    0    0    -1
-$EndComp
 Wire Wire Line
 	8900 4550 8900 4750
@@
 	1    8900 4750
 	1    0    0    -1
-$EndComp
-$Comp
-L Switch:SW_Push SW2
-U 1 1 60F04771
-P 9250 4550
-F 0 "SW2" H 9250 4500 50  0000 C CNN
-F 1 "ARRANQUE" H 9250 4400 50  0000 C CNN
-F 2 "Button_Switch_SMD:SW_SPST_TL3342" H 9250 4743 50  0001 C CNN
-F 3 "https://sten-eswitch-13110800-production.s3.amazonaws.com/system/asset/product_line/data_sheet/165/TL3342.pdf" H 9250 4750 50  0001 C CNN
-	1    9250 4550
-	1    0    0    -1
-$EndComp
-$Comp
-L Device:R R32
-U 1 1 60F0476B
-P 9250 4350
-F 0 "R32" V 9043 4350 50  0000 C CNN
-F 1 "10K" H 9134 4350 50  0000 C CNN
-F 2 "Resistor_SMD:R_0805_2012Metric" V 9180 4350 50  0001 C CNN
-F 3 "~" H 9250 4350 50  0001 C CNN
-	1    9250 4350
-	0    1    1    0
 $EndComp
 Text HLabel 9000 5950 0    50   BiDi ~ 0
@@
 	9050 3300 8900 3300
 Wire Wire Line
-	9100 3100 8900 3100
-Wire Wire Line
-	8900 2850 8900 3100
-$Comp
-L power:+3.3V #PWR0137
-U 1 1 60DFF360
-P 8900 2850
-F 0 "#PWR0137" H 8900 2700 50  0001 C CNN
-F 1 "+3.3V" H 8915 3023 50  0000 C CNN
-F 2 "" H 8900 2850 50  0001 C CNN
-F 3 "" H 8900 2850 50  0001 C CNN
-	1    8900 2850
-	1    0    0    -1
-$EndComp
-Wire Wire Line
 	8900 3300 8900 3500
 $Comp
@@
 	1    9250 3300
 	1    0    0    -1
-$EndComp
-$Comp
-L Device:R R10
-U 1 1 60DDAD0C
-P 9250 3100
-F 0 "R10" V 9043 3100 50  0000 C CNN
-F 1 "10K" H 9134 3100 50  0000 C CNN
-F 2 "Resistor_SMD:R_0805_2012Metric" V 9180 3100 50  0001 C CNN
-F 3 "~" H 9250 3100 50  0001 C CNN
-	1    9250 3100
-	0    1    1    0
 $EndComp
 Text Label 1950 3850 2    50   ~ 0
@@
 	1    0    0    -1
 $EndComp
+$Comp
+L Switch:SW_Push SW2
+U 1 1 60F04771
+P 9250 4550
+F 0 "SW2" H 9250 4500 50  0000 C CNN
+F 1 "ARRANQUE" H 9250 4400 50  0000 C CNN
+F 2 "Button_Switch_SMD:SW_SPST_TL3342" H 9250 4743 50  0001 C CNN
+F 3 "https://sten-eswitch-13110800-production.s3.amazonaws.com/system/asset/product_line/data_sheet/165/TL3342.pdf" H 9250 4750 50  0001 C CNN
+	1    9250 4550
+	1    0    0    -1
+$EndComp
+Connection ~ 9600 4350
+Wire Wire Line
+	9600 4350 9400 4350
+$Comp
+L Device:C C7
+U 1 1 6100DA28
+P 9250 3100
+F 0 "C7" V 9502 3100 50  0000 C CNN
+F 1 "0.1uf" V 9411 3100 50  0000 C CNN
+F 2 "Capacitor_SMD:C_0805_2012Metric" H 9288 2950 50  0001 C CNN
+F 3 "~" H 9250 3100 50  0001 C CNN
+	1    9250 3100
+	0    -1   -1   0
+$EndComp
+$Comp
+L Device:C C8
+U 1 1 610107FF
+P 9250 4350
+F 0 "C8" V 8998 4350 50  0000 C CNN
+F 1 "0.1uf" V 9089 4350 50  0000 C CNN
+F 2 "Capacitor_SMD:C_0805_2012Metric" H 9288 4200 50  0001 C CNN
+F 3 "~" H 9250 4350 50  0001 C CNN
+	1    9250 4350
+	0    1    1    0
+$EndComp
+Wire Wire Line
+	9100 3100 8900 3100
+Wire Wire Line
+	8900 3100 8900 3300
+Connection ~ 8900 3300
+Wire Wire Line
+	9100 4350 8900 4350
+Wire Wire Line
+	8900 4350 8900 4550
+Connection ~ 8900 4550
 $EndSCHEMATC
