File: Control de Gabinetes/comunicacion.sch (KiCad schematic (older format))
At the start: 1 part

Commit message: AVANCE 13/07/2021
Parts:
- removed J?: Conn_01x07_Female, symbol Connector:Conn_01x07_Female
- added AE1: Antenna, RF_Antenna:Texas_SWRA416_868MHz_915MHz, symbol Device:Antenna
- added Q1: PN2222A, Package_TO_SOT_SMD:SOT-23, symbol Transistor_BJT:PN2222A
- added R13, R14: R0, Resistor_SMD:R_0805_2012Metric, symbol Device:R
- added R15: 4.7K, Resistor_SMD:R_0805_2012Metric, symbol Device:R
- added R16: 47K, Resistor_SMD:R_0805_2012Metric, symbol Device:R
- added U4: RF-LORA-915-SO, RF-LORA-868-SO:XCVR_RF-LORA-868-SO, symbol RF-LORA-868-SO:RF-LORA-868-SO
- added U5: SIM7600SA, SIM7600SA:SIM7600SA, symbol SIM7600SA:SIM7600SA
Connections:
- net 3.3V: now also U4.3 (VCC)
- net 5V: now also U5.5 (VCC)
- net CS: now also U4.16 (~SEL)
- net DIO0: now also U4.6 (DIO0)
- net GND: now also Q1.1 (E), R16.1, U4.2 (GND), U5.1 (GND), U5.6 (GND)
- net MISO: now also U4.14 (SDO)
- net MOSI: now also U4.15 (SDI)
- net PWRKEY: now also Q1.3 (C), R15.2, U5.4 (PWRKEY)
- net RESET_L: now also U4.12 (RESET)
- net RX2: now also U5.3 (TX)
- net SCK: now also U4.13 (SCLK)
- net SLEEP1: now also U5.7 (SLEEP)
- net TX2: now also U5.2 (RX)
- new net: AE1.1 (A), U4.1 (ANT)
- new net: R13.1, U4.4 (RX_SWITCH)
- new net: R14.1, U4.5 (TX_SWITCH)
- new net: Q1.2 (B), R15.1, R16.2
- new net RX_SWITCH: R13.2
- new net TX_SWITCH: R14.2
Other:
- note added: "MODULO CELULAR 4G"
- note removed: "MODULO CELULAR"

Commit message: avance2 19/07/2021
Parts:
- added D7, D8: LED, LED_SMD:LED_0805_2012Metric, symbol Device:LED
Connections:
- net GND: now also D7.1 (K), D8.1 (K)
- net PWRKEY: no longer Q1.3 (C), U5.4 (PWRKEY)
- net RX_SWITCH: no longer names the net of R13.2
- net RX_SWITCH: now also D7.2 (A)
- net TX_SWITCH: no longer names the net of R14.2
- net TX_SWITCH: now also D8.2 (A)
- new net POWERKEY: Q1.3 (C), U5.4 (PWRKEY)
Changed lines of the file:
@@
 Text Label 2400 4200 2    50   ~ 0
 MOSI
-Text Label 1800 4100 2    50   ~ 0
+Text Label 2400 4100 2    50   ~ 0
 SCK
 Text Label 2400 3600 2    50   ~ 0
@@
 Wire Wire Line
 	2200 4500 2600 4500
-Text HLabel 1800 3800 0    50   Input ~ 0
-RX_SWITCH
-Text HLabel 1800 3900 0    50   Input ~ 0
-TX_SWITCH
 $Comp
 L SIM7600SA:SIM7600SA U5
@@
 	3200 2050 3650 2050
 Text Label 3200 1750 0    50   ~ 0
-PWRKEY
+POWERKEY
 $Comp
 L Device:R R13
@@
 Wire Wire Line
 	2600 3900 2400 3900
-Wire Wire Line
-	1800 3900 2100 3900
-Wire Wire Line
-	1800 3800 2100 3800
 $Comp
 L Device:Antenna AE1
@@
 GND
 Text Label 2000 1300 0    50   ~ 0
-PWRKEY
+POWERKEY
+$Comp
+L Device:LED D7
+U 1 1 60FDB734
+P 1000 4150
+F 0 "D7" V 1039 4032 50  0000 R CNN
+F 1 "LED" V 948 4032 50  0000 R CNN
+F 2 "LED_SMD:LED_0805_2012Metric" H 1000 4150 50  0001 C CNN
+F 3 "~" H 1000 4150 50  0001 C CNN
+	1    1000 4150
+	0    -1   -1   0
+$EndComp
+$Comp
+L Device:LED D8
+U 1 1 60FDCA55
+P 1350 4150
+F 0 "D8" V 1389 4032 50  0000 R CNN
+F 1 "LED" V 1298 4032 50  0000 R CNN
+F 2 "LED_SMD:LED_0805_2012Metric" H 1350 4150 50  0001 C CNN
+F 3 "~" H 1350 4150 50  0001 C CNN
+	1    1350 4150
+	0    -1   -1   0
+$EndComp
+Wire Wire Line
+	2100 3900 1350 3900
+Wire Wire Line
+	1350 3900 1350 4000
+Wire Wire Line
+	2100 3800 1000 3800
+Wire Wire Line
+	1000 3800 1000 4000
+$Comp
+L power:GND #PWR0146
+U 1 1 60FDFE4A
+P 1000 4500
+F 0 "#PWR0146" H 1000 4250 50  0001 C CNN
+F 1 "GND" H 1005 4327 50  0000 C CNN
+F 2 "" H 1000 4500 50  0001 C CNN
+F 3 "" H 1000 4500 50  0001 C CNN
+	1    1000 4500
+	1    0    0    -1
+$EndComp
+$Comp
+L power:GND #PWR0147
+U 1 1 60FE02F7
+P 1350 4500
+F 0 "#PWR0147" H 1350 4250 50  0001 C CNN
+F 1 "GND" H 1355 4327 50  0000 C CNN
+F 2 "" H 1350 4500 50  0001 C CNN
+F 3 "" H 1350 4500 50  0001 C CNN
+	1    1350 4500
+	1    0    0    -1
+$EndComp
+Wire Wire Line
+	1000 4500 1000 4300
+Wire Wire Line
+	1350 4500 1350 4300
 $EndSCHEMATC

Commit message: avance 20/07/2021
Parts:
- AE1: footprint RF_Antenna:Texas_SWRA416_868MHz_915MHz -> RF-LORA-868-SO:Texas_SWRA416_868MHz_915MHz
Connections:
- net ANT: now reaches AE1.1 (A), U4.1 (ANT)
Changed lines of the file:
@@
 	2200 4300 2600 4300
-Wire Wire Line
-	2200 3600 2600 3600
 Wire Wire Line
 	2100 3500 2600 3500
@@
 Wire Wire Line
 	2600 3900 2400 3900
-$Comp
-L Device:Antenna AE1
-U 1 1 60EE4EBF
-P 4600 4000
-F 0 "AE1" H 4680 3989 50  0000 L CNN
-F 1 "Antenna" H 4680 3898 50  0000 L CNN
-F 2 "RF_Antenna:Texas_SWRA416_868MHz_915MHz" H 4600 4000 50  0001 C CNN
-F 3 "~" H 4600 4000 50  0001 C CNN
-	1    4600 4000
-	1    0    0    -1
-$EndComp
-Wire Wire Line
-	4000 4300 4600 4300
 Wire Wire Line
 	4600 4300 4600 4200
@@
 Wire Wire Line
 	1350 4500 1350 4300
+Wire Wire Line
+	4000 4300 4600 4300
+Wire Wire Line
+	2200 3600 2600 3600
+Text Label 4350 4300 0    50   ~ 0
+ANT
+$Comp
+L Device:Antenna AE1
+U 1 1 60EE4EBF
+P 4600 4000
+F 0 "AE1" H 4680 3989 50  0000 L CNN
+F 1 "Antenna" H 4680 3898 50  0000 L CNN
+F 2 "RF-LORA-868-SO:Texas_SWRA416_868MHz_915MHz" H 4600 4000 50  0001 C CNN
+F 3 "~" H 4600 4000 50  0001 C CNN
+	1    4600 4000
+	1    0    0    -1
+$EndComp
 $EndSCHEMATC
