File: Control de Gabinetes/sensores.sch (KiCad schematic (older format))
At the start: 5 parts

Commit message: Avance 1/07/2021
Parts:
- gave numbers to parts that had none: 5
Changed lines of the file:
@@
 $EndDescr
 $Comp
-L Connector_Generic:Conn_01x03 J?
+L Connector_Generic:Conn_01x03 J3
 U 1 1 609BD109
 P 1550 2350
-F 0 "J?" H 1468 2025 50  0000 C CNN
+F 0 "J3" H 1468 2025 50  0000 C CNN
 F 1 "MOVIMIENTO" H 1468 2116 50  0000 C CNN
 F 2 "Connector_Molex:Molex_KK-254_AE-6410-03A_1x03_P2.54mm_Vertical" H 1550 2350 50  0001 C CNN
@@
 $EndComp
 $Comp
-L Connector_Generic:Conn_01x04 J?
+L Connector_Generic:Conn_01x04 J4
 U 1 1 609BE811
 P 1550 3350
-F 0 "J?" H 1468 2925 50  0000 C CNN
+F 0 "J4" H 1468 2925 50  0000 C CNN
 F 1 "TEMPERATURA PRESION" H 1468 3016 50  0000 C CNN
 F 2 "Connector_Molex:Molex_KK-254_AE-6410-04A_1x04_P2.54mm_Vertical" H 1550 3350 50  0001 C CNN
@@
 $EndComp
 $Comp
-L Connector_Generic:Conn_01x03 J?
+L Connector_Generic:Conn_01x03 J5
 U 1 1 609BF6A2
 P 1550 4350
-F 0 "J?" H 1468 4025 50  0000 C CNN
+F 0 "J5" H 1468 4025 50  0000 C CNN
 F 1 "HUMEDAD" H 1468 4116 50  0000 C CNN
 F 2 "Connector_Molex:Molex_KK-254_AE-6410-03A_1x03_P2.54mm_Vertical" H 1550 4350 50  0001 C CNN
@@
 $EndComp
 $Comp
-L Connector_Generic:Conn_01x02 J?
+L Connector_Generic:Conn_01x02 J2
 U 1 1 609C0797
 P 1550 1450
-F 0 "J?" H 1468 1125 50  0000 C CNN
+F 0 "J2" H 1468 1125 50  0000 C CNN
 F 1 "APERTURA" H 1468 1216 50  0000 C CNN
 F 2 "Connector_Molex:Molex_KK-254_AE-6410-02A_1x02_P2.54mm_Vertical" H 1550 1450 50  0001 C CNN
@@
 $EndComp
 $Comp
-L power:+5V #PWR?
+L power:+5V #PWR0114
 U 1 1 609C13BA
 P 1950 2450
-F 0 "#PWR?" H 1950 2300 50  0001 C CNN
-F 1 "+5V" H 1965 2623 50  0000 C CNN
+F 0 "#PWR0114" H 1950 2300 50  0001 C CNN
+F 1 "+5V" V 1950 2650 50  0000 C CNN
 F 2 "" H 1950 2450 50  0001 C CNN
 F 3 "" H 1950 2450 50  0001 C CNN
@@
 $EndComp
 $Comp
-L power:+5V #PWR?
+L power:+5V #PWR0115
 U 1 1 609C387F
 P 1950 4450
-F 0 "#PWR?" H 1950 4300 50  0001 C CNN
+F 0 "#PWR0115" H 1950 4300 50  0001 C CNN
 F 1 "+5V" V 1965 4578 50  0000 L CNN
 F 2 "" H 1950 4450 50  0001 C CNN
@@
 $EndComp
 Wire Wire Line
-	1750 2450 1950 2450
-$Comp
-L power:+3.3V #PWR?
+	1750 2450 1850 2450
+$Comp
+L power:+3.3V #PWR0116
 U 1 1 609C4E7A
 P 1950 3450
-F 0 "#PWR?" H 1950 3300 50  0001 C CNN
+F 0 "#PWR0116" H 1950 3300 50  0001 C CNN
 F 1 "+3.3V" V 1965 3578 50  0000 L CNN
 F 2 "" H 1950 3450 50  0001 C CNN
@@
 $EndComp
 $Comp
-L power:GND #PWR?
+L power:GND #PWR0117
 U 1 1 609C56AF
 P 1950 3350
-F 0 "#PWR?" H 1950 3100 50  0001 C CNN
+F 0 "#PWR0117" H 1950 3100 50  0001 C CNN
 F 1 "GND" V 1955 3222 50  0000 R CNN
 F 2 "" H 1950 3350 50  0001 C CNN
@@
 $EndComp
 Wire Wire Line
-	1950 3250 1750 3250
-Wire Wire Line
-	1950 3150 1750 3150
-Wire Wire Line
 	1750 3350 1950 3350
-Wire Wire Line
-	1950 3450 1750 3450
 Text Label 1950 3250 0    50   ~ 0
 SCL
@@
 	1950 4450 1750 4450
 $Comp
-L power:GND #PWR?
+L power:GND #PWR0118
 U 1 1 609C6D05
 P 1950 4250
-F 0 "#PWR?" H 1950 4000 50  0001 C CNN
+F 0 "#PWR0118" H 1950 4000 50  0001 C CNN
 F 1 "GND" V 1955 4122 50  0000 R CNN
 F 2 "" H 1950 4250 50  0001 C CNN
@@
 $EndComp
 $Comp
-L power:+3.3V #PWR?
+L power:+3.3V #PWR0119
 U 1 1 609C79F6
 P 1950 1450
-F 0 "#PWR?" H 1950 1300 50  0001 C CNN
+F 0 "#PWR0119" H 1950 1300 50  0001 C CNN
 F 1 "+3.3V" V 1965 1578 50  0000 L CNN
 F 2 "" H 1950 1450 50  0001 C CNN
@@
 	0    1    1    0
 $EndComp
-Wire Wire Line
-	1950 1450 1750 1450
 Text Label 1950 4350 0    50   ~ 0
 S_HUMEDAD
 $Comp
-L power:GND #PWR?
+L power:GND #PWR0120
 U 1 1 609C86DA
 P 1950 2250
-F 0 "#PWR?" H 1950 2000 50  0001 C CNN
+F 0 "#PWR0120" H 1950 2000 50  0001 C CNN
 F 1 "GND" V 1955 2122 50  0000 R CNN
 F 2 "" H 1950 2250 50  0001 C CNN
@@
 	1950 1350 1750 1350
 Wire Wire Line
-	2650 1350 2450 1350
-$Comp
-L power:GND #PWR?
+	2650 1350 2550 1350
+$Comp
+L power:GND #PWR0121
 U 1 1 609CFF9B
 P 2650 1350
-F 0 "#PWR?" H 2650 1100 50  0001 C CNN
+F 0 "#PWR0121" H 2650 1100 50  0001 C CNN
 F 1 "GND" V 2655 1222 50  0000 R CNN
 F 2 "" H 2650 1350 50  0001 C CNN
@@
 $EndComp
 $Comp
-L Device:R R?
+L Device:R R1
 U 1 1 609CB315
 P 2300 1350
-F 0 "R?" V 2507 1350 50  0000 C CNN
+F 0 "R1" V 2507 1350 50  0000 C CNN
 F 1 "10K" V 2416 1350 50  0000 C CNN
 F 2 "Resistor_SMD:R_0805_2012Metric" V 2230 1350 50  0001 C CNN
@@
 Text Label 1950 1150 0    50   ~ 0
 S_APERTURA
+Wire Wire Line
+	1950 1450 1850 1450
+Wire Wire Line
+	2000 1550 1850 1550
+Wire Wire Line
+	1850 1550 1850 1450
+Connection ~ 1850 1450
+Wire Wire Line
+	1850 1450 1750 1450
+Wire Wire Line
+	2000 2550 1850 2550
+Wire Wire Line
+	1850 2550 1850 2450
+Connection ~ 1850 2450
+Wire Wire Line
+	1850 2450 1950 2450
+Text HLabel 2000 2550 2    50   Input ~ 0
+5V
+Wire Wire Line
+	1750 3450 1950 3450
+Text HLabel 2000 1550 2    50   Input ~ 0
+3.3V
+Text HLabel 2700 1450 2    50   Input ~ 0
+GND
+Wire Wire Line
+	2700 1450 2550 1450
+Wire Wire Line
+	2550 1450 2550 1350
+Connection ~ 2550 1350
+Wire Wire Line
+	2550 1350 2450 1350
+Wire Wire Line
+	1750 3150 2200 3150
+Wire Wire Line
+	1750 3250 2200 3250
+Text HLabel 2200 3150 2    50   BiDi ~ 0
+SDA
+Text HLabel 2200 3250 2    50   BiDi ~ 0
+SCL
 $EndSCHEMATC

Commit message: avance 6/07
Parts:
- added R? (x3): 10K, Resistor_SMD:R_0805_2012Metric, symbol Device:R
- added R?: 20K, Resistor_SMD:R_0805_2012Metric, symbol Device:R
Connections:
- net GND: now also R?.2, R?.2
- net S_HUMEDAD: now also R?.1, R?.2; no longer J5.2 (Pin_2)
- net S_MOVIMIENTO: now also R?.1, R?.2; no longer J3.2 (Pin_2)
- new net: J3.2 (Pin_2), R?.1
- new net: J5.2 (Pin_2), R?.1
Other:
- note added: "ENTRADA DIGITAL: SENSOR DE MOVIMIENTO\n"
- note added: "ENTRADA DIGITAL: SENSOR DHT11"
- note added: "ENTRADA DIGITAL: SENSOR MAGNETICO\n"
- note added: "ENTRADA I2C: SENSOR BPN280"
- moved on the sheet: J2, J3, J4, J5, R1

Commit message: AVANCE 13/07/2021
Parts:
- gave numbers to parts that had none: 4
Changed lines of the file:
@@
 ENTRADA DIGITAL: SENSOR DHT11
 $Comp
-L Device:R R?
+L Device:R R7
 U 1 1 60E439CB
 P 2850 2550
-F 0 "R?" V 3057 2550 50  0000 C CNN
+F 0 "R7" V 3057 2550 50  0000 C CNN
 F 1 "10K" V 2966 2550 50  0000 C CNN
 F 2 "Resistor_SMD:R_0805_2012Metric" V 2780 2550 50  0001 C CNN
@@
 	3000 2550 3150 2550
 $Comp
-L Device:R R?
+L Device:R R8
 U 1 1 60E44296
 P 3450 2550
-F 0 "R?" V 3657 2550 50  0000 C CNN
+F 0 "R8" V 3657 2550 50  0000 C CNN
 F 1 "20K" V 3566 2550 50  0000 C CNN
 F 2 "Resistor_SMD:R_0805_2012Metric" V 3380 2550 50  0001 C CNN
@@
 	3600 2550 3800 2550
 $Comp
-L power:GND #PWR?
+L power:GND #PWR0130
 U 1 1 60E48F01
 P 3800 2550
-F 0 "#PWR?" H 3800 2300 50  0001 C CNN
+F 0 "#PWR0130" H 3800 2300 50  0001 C CNN
 F 1 "GND" V 3805 2422 50  0000 R CNN
 F 2 "" H 3800 2550 50  0001 C CNN
@@
 S_APERTURA
 $Comp
-L Device:R R?
+L Device:R R6
 U 1 1 60E5FD52
 P 2800 4550
-F 0 "R?" V 3007 4550 50  0000 C CNN
+F 0 "R6" V 3007 4550 50  0000 C CNN
 F 1 "10K" V 2916 4550 50  0000 C CNN
 F 2 "Resistor_SMD:R_0805_2012Metric" V 2730 4550 50  0001 C CNN
@@
 $EndComp
 $Comp
-L Device:R R?
+L Device:R R9
 U 1 1 60E605A2
 P 3500 4550
-F 0 "R?" V 3707 4550 50  0000 C CNN
+F 0 "R9" V 3707 4550 50  0000 C CNN
 F 1 "10K" V 3616 4550 50  0000 C CNN
 F 2 "Resistor_SMD:R_0805_2012Metric" V 3430 4550 50  0001 C CNN
@@
 	3350 4550 3150 4550
 $Comp
-L power:GND #PWR?
+L power:GND #PWR0131
 U 1 1 60E61546
 P 3850 4550
-F 0 "#PWR?" H 3850 4300 50  0001 C CNN
+F 0 "#PWR0131" H 3850 4300 50  0001 C CNN
 F 1 "GND" V 3855 4422 50  0000 R CNN
 F 2 "" H 3850 4550 50  0001 C CNN
