File: Control de Gabinetes/actuadores.sch (KiCad schematic (older format))
At the start: 0 parts

Commit message: avance 19/07
Parts:
- added D3, D4, D5, D6: US1J, Diode_SMD:D_SMA, symbol Diode:US1J
- added J10, J7, J8, J9: Screw_Terminal_01x02, TerminalBlock:TerminalBlock_bornier-2_P5.08mm, symbol Connector:Screw_Terminal_01x02
- added K1, K2, K3, K4: FINDER-36.11, Relay_THT:Relay_SPDT_Finder_36.11, symbol Relay:FINDER-36.11
- added Q2, Q3, Q4, Q5: PN2222A, Package_TO_SOT_THT:TO-92_Inline, symbol Transistor_BJT:PN2222A
- added R17, R18, R19, R20: 500, Resistor_SMD:R_0805_2012Metric, symbol Device:R
- added R21, R22, R23, R24: 2.2K, Resistor_SMD:R_0805_2012Metric, symbol Device:R
- added R25, R26, R27, R28: 10K, Resistor_SMD:R_0805_2012Metric, symbol Device:R
- added U6, U7, U8, U9: SFH6156-2T, SOT254P978X405-4N, symbol SFH6156-2T:SFH6156-2T
Connections:
- new net: Q2.2 (B), R25.1
- new net: D3.2 (A), K1.A2, Q2.3 (C)
- new net: R17.1, U6.1
- new net: R21.2, R25.2, U6.3
- new net: Q3.2 (B), R26.1
- new net: D4.2 (A), K2.A2, Q3.3 (C)
- new net: R18.1, U7.1
- new net: R22.2, R26.2, U7.3
- new net: Q4.2 (B), R27.1
- new net: D5.2 (A), K3.A2, Q4.3 (C)
- new net: R19.1, U8.1
- new net: R23.2, R27.2, U8.3
- new net: Q5.2 (B), R28.1
- new net: D6.2 (A), K4.A2, Q5.3 (C)
- new net: R20.1, U9.1
- new net: R24.2, R28.2, U9.3
- new net 5V: D3.1 (K), D4.1 (K), D5.1 (K), D6.1 (K), K1.A1, K2.A1, K3.A1, K4.A1, U6.4, U7.4, U8.4, U9.4
- new net GND: Q2.1 (E), Q3.1 (E), Q4.1 (E), Q5.1 (E), R22.1, R23.1, R24.1, U6.2, U7.2, U8.2, U9.2
- new net LINEA1: J7.2 (Pin_2), K1.11
- new net LINEA1_CARGA: J7.1 (Pin_1), K1.14
- new net LINEA2: J8.2 (Pin_2), K2.11
- new net LINEA2_CARGA: J8.1 (Pin_1), K2.14
- new net LINEA3: J9.2 (Pin_2), K3.11
- new net LINEA3_CARGA: J9.1 (Pin_1), K3.14
- new net LINEA4: J10.2 (Pin_2), K4.11
- new net LINEA4_CARGA: J10.1 (Pin_1), K4.14
- new net RELAY1: R17.2, R18.2, R19.2, R20.2
