File: Control de Gabinetes/actuadores.sch (KiCad schematic (older format))
At the start: 32 parts, among them J10 Screw_Terminal_01x02, J7 Screw_Terminal_01x02, J8 Screw_Terminal_01x02, J9 Screw_Terminal_01x02, K1 FINDER-36.11, K2 FINDER-36.11, K3 FINDER-36.11, K4 FINDER-36.11, Q2 PN2222A, Q3 PN2222A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

Commit message: avance2 19/07/2021
Parts:
- Q2, Q3, Q4, Q5: footprint Package_TO_SOT_THT:TO-92_Inline -> Package_TO_SOT_SMD:SOT-23
Connections:
- net RELAY1: no longer R18.2, R19.2, R20.2
- new net RELAY2: R18.2
- new net RELAY3: R19.2
- new net RELAY4: R20.2
Other:
- note added: "ACTUADORES"
Changed lines of the file:
@@
 F 0 "Q2" H 5290 2346 50  0000 L CNN
 F 1 "PN2222A" H 5290 2255 50  0000 L CNN
-F 2 "Package_TO_SOT_THT:TO-92_Inline" H 5300 2225 50  0001 L CIN
+F 2 "Package_TO_SOT_SMD:SOT-23" H 5300 2225 50  0001 L CIN
 F 3 "https://www.onsemi.com/pub/Collateral/PN2222-D.PDF" H 5100 2300 50  0001 L CNN
 	1    5100 2300
@@
 F 0 "Q3" H 5290 4846 50  0000 L CNN
 F 1 "PN2222A" H 5290 4755 50  0000 L CNN
-F 2 "Package_TO_SOT_THT:TO-92_Inline" H 5300 4725 50  0001 L CIN
+F 2 "Package_TO_SOT_SMD:SOT-23" H 5300 4725 50  0001 L CIN
 F 3 "https://www.onsemi.com/pub/Collateral/PN2222-D.PDF" H 5100 4800 50  0001 L CNN
 	1    5100 4800
@@
 	2200 4500 2600 4500
 Text Label 2350 4500 0    50   ~ 0
-RELAY1
+RELAY2
 Text HLabel 2200 4500 0    50   Input ~ 0
 RELAY2
@@
 F 0 "Q4" H 5290 7296 50  0000 L CNN
 F 1 "PN2222A" H 5290 7205 50  0000 L CNN
-F 2 "Package_TO_SOT_THT:TO-92_Inline" H 5300 7175 50  0001 L CIN
+F 2 "Package_TO_SOT_SMD:SOT-23" H 5300 7175 50  0001 L CIN
 F 3 "https://www.onsemi.com/pub/Collateral/PN2222-D.PDF" H 5100 7250 50  0001 L CNN
 	1    5100 7250
@@
 	2200 6950 2600 6950
 Text Label 2350 6950 0    50   ~ 0
-RELAY1
+RELAY3
 Text HLabel 2200 6950 0    50   Input ~ 0
 RELAY3
@@
 F 0 "Q5" H 5290 9796 50  0000 L CNN
 F 1 "PN2222A" H 5290 9705 50  0000 L CNN
-F 2 "Package_TO_SOT_THT:TO-92_Inline" H 5300 9675 50  0001 L CIN
+F 2 "Package_TO_SOT_SMD:SOT-23" H 5300 9675 50  0001 L CIN
 F 3 "https://www.onsemi.com/pub/Collateral/PN2222-D.PDF" H 5100 9750 50  0001 L CNN
 	1    5100 9750
@@
 	2200 9450 2600 9450
 Text Label 2350 9450 0    50   ~ 0
-RELAY1
+RELAY4
 Text HLabel 2200 9450 0    50   Input ~ 0
 RELAY4
@@
 	2800 7250 2900 7250
 Connection ~ 2900 7250
+Text Notes 4700 800  0    79   ~ 0
+ACTUADORES
 $EndSCHEMATC

Commit message: avance 20/07/2021
Parts:
- J10, J7, J8, J9: footprint TerminalBlock:TerminalBlock_bornier-2_P5.08mm -> TerminalBlockjuan:TerminalBlock_bornier-2_P5.08mm
Connections:
- net GND: now also R21.1
Changed lines of the file:
@@
 L power:GND #PWR0123
 U 1 1 60F70F7A
-P 4200 2950
-F 0 "#PWR0123" H 4200 2700 50  0001 C CNN
-F 1 "GND" H 4205 2777 50  0000 C CNN
-F 2 "" H 4200 2950 50  0001 C CNN
-F 3 "" H 4200 2950 50  0001 C CNN
-	1    4200 2950
+P 4200 2900
+F 0 "#PWR0123" H 4200 2650 50  0001 C CNN
+F 1 "GND" H 4205 2727 50  0000 C CNN
+F 2 "" H 4200 2900 50  0001 C CNN
+F 3 "" H 4200 2900 50  0001 C CNN
+	1    4200 2900
 	1    0    0    -1
 $EndComp
@@
 F 0 "J7" H 6680 1492 50  0000 L CNN
 F 1 "Screw_Terminal_01x02" H 6680 1401 50  0000 L CNN
-F 2 "TerminalBlock:TerminalBlock_bornier-2_P5.08mm" H 6600 1500 50  0001 C CNN
+F 2 "TerminalBlockjuan:TerminalBlock_bornier-2_P5.08mm" H 6600 1500 50  0001 C CNN
 F 3 "~https://www.didacticaselectronicas.com/index.php/suiches-y-conectores/borneras/bornera-2p-verde-kf128-5mm-kf128-2p-borneras-terminales-con-borneras-screw-terminal-terminal-block-de-2-pines-2-posiciones-kf128-5mm-detail" H 6600 1500 50  0001 C CNN
 	1    6600 1500
@@
 F 0 "J8" H 6680 3992 50  0000 L CNN
 F 1 "Screw_Terminal_01x02" H 6680 3901 50  0000 L CNN
-F 2 "TerminalBlock:TerminalBlock_bornier-2_P5.08mm" H 6600 4000 50  0001 C CNN
+F 2 "TerminalBlockjuan:TerminalBlock_bornier-2_P5.08mm" H 6600 4000 50  0001 C CNN
 F 3 "~https://www.didacticaselectronicas.com/index.php/suiches-y-conectores/borneras/bornera-2p-verde-kf128-5mm-kf128-2p-borneras-terminales-con-borneras-screw-terminal-terminal-block-de-2-pines-2-posiciones-kf128-5mm-detail" H 6600 4000 50  0001 C CNN
 	1    6600 4000
@@
 F 0 "J9" H 6680 6442 50  0000 L CNN
 F 1 "Screw_Terminal_01x02" H 6680 6351 50  0000 L CNN
-F 2 "TerminalBlock:TerminalBlock_bornier-2_P5.08mm" H 6600 6450 50  0001 C CNN
+F 2 "TerminalBlockjuan:TerminalBlock_bornier-2_P5.08mm" H 6600 6450 50  0001 C CNN
 F 3 "~https://www.didacticaselectronicas.com/index.php/suiches-y-conectores/borneras/bornera-2p-verde-kf128-5mm-kf128-2p-borneras-terminales-con-borneras-screw-terminal-terminal-block-de-2-pines-2-posiciones-kf128-5mm-detail" H 6600 6450 50  0001 C CNN
 	1    6600 6450
@@
 F 0 "J10" H 6680 8942 50  0000 L CNN
 F 1 "Screw_Terminal_01x02" H 6680 8851 50  0000 L CNN
-F 2 "TerminalBlock:TerminalBlock_bornier-2_P5.08mm" H 6600 8950 50  0001 C CNN
+F 2 "TerminalBlockjuan:TerminalBlock_bornier-2_P5.08mm" H 6600 8950 50  0001 C CNN
 F 3 "~https://www.didacticaselectronicas.com/index.php/suiches-y-conectores/borneras/bornera-2p-verde-kf128-5mm-kf128-2p-borneras-terminales-con-borneras-screw-terminal-terminal-block-de-2-pines-2-posiciones-kf128-5mm-detail" H 6600 8950 50  0001 C CNN
 	1    6600 8950
