File: Control de Gabinetes/Control de Gabinetes.sch (KiCad schematic (older format))
At the start: 0 parts

Commit message: Avance 1/07/2021
Changed lines of the file:
@@
 F0 "regulacion" 50
 F1 "regulacion.sch" 50
+F2 "3.3V" O L 1600 1900 50
+F3 "5V" O L 1600 1800 50
+F4 "12V" O L 1600 1700 50
+F5 "GND" O L 1600 2000 50
 $EndSheet
 $Sheet
@@
 F0 "sensores" 50
 F1 "sensores.sch" 50
+F2 "5V" I L 1750 4300 50
+F3 "3.3V" I L 1750 4400 50
+F4 "GND" I L 1750 4500 50
+F5 "SDA" B L 1750 4600 50
+F6 "SCL" B L 1750 4700 50
 $EndSheet
 $Sheet
@@
 F1 "comunicacion.sch" 50
 $EndSheet
+$Comp
+L power:+12V #PWR0101
+U 1 1 60A32ADA
+P 1400 1700
+F 0 "#PWR0101" H 1400 1550 50  0001 C CNN
+F 1 "+12V" V 1415 1828 50  0000 L CNN
+F 2 "" H 1400 1700 50  0001 C CNN
+F 3 "" H 1400 1700 50  0001 C CNN
+	1    1400 1700
+	0    -1   -1   0
+$EndComp
+$Comp
+L power:+5V #PWR0102
+U 1 1 60A336D2
+P 1400 1800
+F 0 "#PWR0102" H 1400 1650 50  0001 C CNN
+F 1 "+5V" V 1415 1928 50  0000 L CNN
+F 2 "" H 1400 1800 50  0001 C CNN
+F 3 "" H 1400 1800 50  0001 C CNN
+	1    1400 1800
+	0    -1   -1   0
+$EndComp
+$Comp
+L power:+3.3V #PWR0103
+U 1 1 60A33DC4
+P 1400 1900
+F 0 "#PWR0103" H 1400 1750 50  0001 C CNN
+F 1 "+3.3V" V 1415 2028 50  0000 L CNN
+F 2 "" H 1400 1900 50  0001 C CNN
+F 3 "" H 1400 1900 50  0001 C CNN
+	1    1400 1900
+	0    -1   -1   0
+$EndComp
+Wire Wire Line
+	1400 1700 1600 1700
+Wire Wire Line
+	1600 1800 1400 1800
+Wire Wire Line
+	1400 1900 1600 1900
+$Comp
+L power:+5V #PWR0104
+U 1 1 60A35C39
+P 1550 4300
+F 0 "#PWR0104" H 1550 4150 50  0001 C CNN
+F 1 "+5V" V 1565 4428 50  0000 L CNN
+F 2 "" H 1550 4300 50  0001 C CNN
+F 3 "" H 1550 4300 50  0001 C CNN
+	1    1550 4300
+	0    -1   -1   0
+$EndComp
+$Comp
+L power:+3.3V #PWR0105
+U 1 1 60A35C3F
+P 1550 4400
+F 0 "#PWR0105" H 1550 4250 50  0001 C CNN
+F 1 "+3.3V" V 1565 4528 50  0000 L CNN
+F 2 "" H 1550 4400 50  0001 C CNN
+F 3 "" H 1550 4400 50  0001 C CNN
+	1    1550 4400
+	0    -1   -1   0
+$EndComp
+Wire Wire Line
+	1750 4300 1550 4300
+Wire Wire Line
+	1550 4400 1750 4400
+$Comp
+L power:GND #PWR?
+U 1 1 60DD420E
+P 1400 2000
+F 0 "#PWR?" H 1400 1750 50  0001 C CNN
+F 1 "GND" V 1405 1872 50  0000 R CNN
+F 2 "" H 1400 2000 50  0001 C CNN
+F 3 "" H 1400 2000 50  0001 C CNN
+	1    1400 2000
+	0    1    1    0
+$EndComp
+Wire Wire Line
+	1600 2000 1400 2000
+$Comp
+L power:GND #PWR?
+U 1 1 60DD5651
+P 1550 4500
+F 0 "#PWR?" H 1550 4250 50  0001 C CNN
+F 1 "GND" V 1555 4372 50  0000 R CNN
+F 2 "" H 1550 4500 50  0001 C CNN
+F 3 "" H 1550 4500 50  0001 C CNN
+	1    1550 4500
+	0    1    1    0
+$EndComp
+Wire Wire Line
+	1750 4500 1550 4500
+Wire Wire Line
+	1550 4600 1750 4600
+Wire Wire Line
+	1550 4700 1750 4700
+Text Label 1550 4600 2    50   ~ 0
+SDA
+Text Label 1550 4700 2    50   ~ 0
+SCL
 $EndSCHEMATC

Commit message: avance 6/07
Connections:
- net labels added: S_APERTURA, S_HUMEDAD, S_MOVIMIENTO
- wire segments 9 -> 20
Changed lines of the file:
@@
 $EndDescr
-$Sheet
-S 4550 1050 1550 2250
-U 60989480
-F0 "esp32" 50
-F1 "esp32.sch" 50
-$EndSheet
 $Sheet
 S 1600 1450 1300 1400
@@
 F5 "SDA" B L 1750 4600 50
 F6 "SCL" B L 1750 4700 50
+F7 "S_HUMEDAD" O L 1750 4800 50
+F8 "S_MOVIMIENTO" O L 1750 4900 50
+F9 "S_APERTURA" O L 1750 5000 50
 $EndSheet
 $Sheet
@@
 Text Label 1550 4700 2    50   ~ 0
 SCL
+Wire Wire Line
+	1550 4800 1750 4800
+Wire Wire Line
+	1550 4900 1750 4900
+Wire Wire Line
+	1550 5000 1750 5000
+Text Label 1550 4800 2    50   ~ 0
+S_HUMEDAD
+Text Label 1550 4900 2    50   ~ 0
+S_MOVIMIENTO
+Text Label 1550 5000 2    50   ~ 0
+S_APERTURA
+$Comp
+L power:+5V #PWR?
+U 1 1 60E5F3D9
+P 4350 1300
+F 0 "#PWR?" H 4350 1150 50  0001 C CNN
+F 1 "+5V" V 4365 1428 50  0000 L CNN
+F 2 "" H 4350 1300 50  0001 C CNN
+F 3 "" H 4350 1300 50  0001 C CNN
+	1    4350 1300
+	0    -1   -1   0
+$EndComp
+$Comp
+L power:+3.3V #PWR?
+U 1 1 60E5F3DF
+P 4350 1400
+F 0 "#PWR?" H 4350 1250 50  0001 C CNN
+F 1 "+3.3V" V 4365 1528 50  0000 L CNN
+F 2 "" H 4350 1400 50  0001 C CNN
+F 3 "" H 4350 1400 50  0001 C CNN
+	1    4350 1400
+	0    -1   -1   0
+$EndComp
+Wire Wire Line
+	4550 1300 4350 1300
+Wire Wire Line
+	4350 1400 4550 1400
+$Comp
+L power:GND #PWR?
+U 1 1 60E5F3E7
+P 4350 1500
+F 0 "#PWR?" H 4350 1250 50  0001 C CNN
+F 1 "GND" V 4355 1372 50  0000 R CNN
+F 2 "" H 4350 1500 50  0001 C CNN
+F 3 "" H 4350 1500 50  0001 C CNN
+	1    4350 1500
+	0    1    1    0
+$EndComp
+Wire Wire Line
+	4550 1500 4350 1500
+Wire Wire Line
+	4350 1600 4550 1600
+Wire Wire Line
+	4350 1700 4550 1700
+Text Label 4350 1600 2    50   ~ 0
+SDA
+Text Label 4350 1700 2    50   ~ 0
+SCL
+Wire Wire Line
+	4350 1800 4550 1800
+Wire Wire Line
+	4350 1900 4550 1900
+Wire Wire Line
+	4350 2000 4550 2000
+Text Label 4350 1800 2    50   ~ 0
+S_HUMEDAD
+Text Label 4350 1900 2    50   ~ 0
+S_MOVIMIENTO
+Text Label 4350 2000 2    50   ~ 0
+S_APERTURA
+$Sheet
+S 4550 1050 1550 2250
+U 60989480
+F0 "esp32" 50
+F1 "esp32.sch" 50
+F2 "3.3V" I L 4550 1400 50
+F3 "GND" I L 4550 1500 50
+F4 "SDA" B L 4550 1600 50
+F5 "SCL" B L 4550 1700 50
+F6 "S_HUMEDAD" I L 4550 1800 50
+F7 "S_MOVIMIENTO" I L 4550 1900 50
+F8 "S_APERTURA" I L 4550 2000 50
+$EndSheet
 $EndSCHEMATC

Commit message: AVANCE 7/7/2021
Connections:
- net labels added: CS, DIO0, MISO, MOSI, PWRKEY, RESET_L, RX2, SCK, SLEEP1, TX2
- wire segments 20 -> 43
Changed lines of the file:
@@
 F1 "actuadores.sch" 50
-$EndSheet
-$Sheet
-S 7250 4050 1450 1600
-U 609895D7
-F0 "comunicacion" 50
-F1 "comunicacion.sch" 50
 $EndSheet
 $Comp
@@
 F7 "S_MOVIMIENTO" I L 4550 1900 50
 F8 "S_APERTURA" I L 4550 2000 50
+F9 "RX2" I L 4550 2100 50
+F10 "TX2" O L 4550 2200 50
+F11 "PWRKEY" O L 4550 2300 50
+F12 "SLEEP1" O L 4550 2400 50
+F13 "RESET_L" O L 4550 2500 50
+F14 "SCK" B L 4550 2600 50
+F15 "MISO" I L 4550 2700 50
+F16 "MOSI" O L 4550 2800 50
+F17 "CS" O L 4550 2900 50
+F18 "DIO0" O L 4550 3000 50
 $EndSheet
+Wire Wire Line
+	7000 4450 7200 4450
+Wire Wire Line
+	7000 4550 7200 4550
+Wire Wire Line
+	7000 4650 7200 4650
+Wire Wire Line
+	7000 4750 7200 4750
+Wire Wire Line
+	7000 4850 7200 4850
+Wire Wire Line
+	7000 4950 7200 4950
+Wire Wire Line
+	7000 5050 7200 5050
+$Comp
+L power:+3.3V #PWR?
+U 1 1 60E895C7
+P 7000 4550
+F 0 "#PWR?" H 7000 4400 50  0001 C CNN
+F 1 "+3.3V" V 7015 4678 50  0000 L CNN
+F 2 "" H 7000 4550 50  0001 C CNN
+F 3 "" H 7000 4550 50  0001 C CNN
+	1    7000 4550
+	0    -1   -1   0
+$EndComp
+$Comp
+L power:+5V #PWR?
+U 1 1 60E8A1FB
+P 7000 4450
+F 0 "#PWR?" H 7000 4300 50  0001 C CNN
+F 1 "+5V" V 7015 4578 50  0000 L CNN
+F 2 "" H 7000 4450 50  0001 C CNN
+F 3 "" H 7000 4450 50  0001 C CNN
+	1    7000 4450
+	0    -1   -1   0
+$EndComp
+$Comp
+L power:GND #PWR?
+U 1 1 60E8BB2F
+P 7000 4650
+F 0 "#PWR?" H 7000 4400 50  0001 C CNN
+F 1 "GND" V 7005 4522 50  0000 R CNN
+F 2 "" H 7000 4650 50  0001 C CNN
+F 3 "" H 7000 4650 50  0001 C CNN
+	1    7000 4650
+	0    1    1    0
+$EndComp
+Text Label 7000 4750 2    50   ~ 0
+RX2
+Text Label 7000 4850 2    50   ~ 0
+TX2
+Text Label 7000 4950 2    50   ~ 0
+PWRKEY
+Text Label 7000 5050 2    50   ~ 0
+SLEEP1
+$Sheet
+S 7200 4100 1400 2150
+U 609895D7
+F0 "comunicacion" 50
+F1 "comunicacion.sch" 50
+F2 "GND" B L 7200 4650 50
+F3 "RX2" O L 7200 4750 50
+F4 "TX2" I L 7200 4850 50
+F5 "PWRKEY" I L 7200 4950 50
+F6 "5V" B L 7200 4450 50
+F7 "SLEEP1" I L 7200 5050 50
+F8 "3.3V" B L 7200 4550 50
+F9 "DIO0" B L 7200 5150 50
+F10 "RESET_L" B L 7200 5250 50
+F11 "MISO" B L 7200 5350 50
+F12 "MOSI" B L 7200 5450 50
+F13 "SCK" B L 7200 5550 50
+F14 "CS" B L 7200 5650 50
+$EndSheet
+Wire Wire Line
+	4350 2100 4550 2100
+Wire Wire Line
+	4350 2200 4550 2200
+Wire Wire Line
+	4350 2300 4550 2300
+Wire Wire Line
+	4350 2400 4550 2400
+Text Label 4350 2100 2    50   ~ 0
+RX2
+Text Label 4350 2200 2    50   ~ 0
+TX2
+Text Label 4350 2300 2    50   ~ 0
+PWRKEY
+Text Label 4350 2400 2    50   ~ 0
+SLEEP1
+Wire Wire Line
+	7000 5150 7200 5150
+Wire Wire Line
+	7000 5250 7200 5250
+Wire Wire Line
+	7000 5350 7200 5350
+Wire Wire Line
+	7000 5450 7200 5450
+Wire Wire Line
+	7000 5550 7200 5550
+Wire Wire Line
+	7000 5650 7200 5650
+Text Label 7000 5150 2    50   ~ 0
+DIO0
+Text Label 7000 5250 2    50   ~ 0
+RESET_L
+Text Label 7000 5350 2    50   ~ 0
+MISO
+Text Label 7000 5450 2    50   ~ 0
+MOSI
+Text Label 7000 5550 2    50   ~ 0
+SCK
+Text Label 7000 5650 2    50   ~ 0
+CS
+Wire Wire Line
+	4350 2500 4550 2500
+Text Label 4350 2500 2    50   ~ 0
+RESET_L
+Wire Wire Line
+	4350 2600 4550 2600
+Wire Wire Line
+	4350 2700 4550 2700
+Wire Wire Line
+	4350 2800 4550 2800
+Wire Wire Line
+	4350 2900 4550 2900
+Text Label 4350 2600 2    50   ~ 0
+SCK
+Text Label 4350 2700 2    50   ~ 0
+MISO
+Text Label 4350 2800 2    50   ~ 0
+MOSI
+Text Label 4350 2900 2    50   ~ 0
+CS
+Wire Wire Line
+	4350 3000 4550 3000
+Text Label 4350 3000 2    50   ~ 0
+DIO0
 $EndSCHEMATC

Commit message: AVANCE 13/07/2021
Changed lines of the file:
@@
 	1550 4400 1750 4400
 $Comp
-L power:GND #PWR?
+L power:GND #PWR0122
 U 1 1 60DD420E
 P 1400 2000
-F 0 "#PWR?" H 1400 1750 50  0001 C CNN
+F 0 "#PWR0122" H 1400 1750 50  0001 C CNN
 F 1 "GND" V 1405 1872 50  0000 R CNN
 F 2 "" H 1400 2000 50  0001 C CNN
@@
 	1600 2000 1400 2000
 $Comp
-L power:GND #PWR?
+L power:GND #PWR0123
 U 1 1 60DD5651
 P 1550 4500
-F 0 "#PWR?" H 1550 4250 50  0001 C CNN
+F 0 "#PWR0123" H 1550 4250 50  0001 C CNN
 F 1 "GND" V 1555 4372 50  0000 R CNN
 F 2 "" H 1550 4500 50  0001 C CNN
@@
 S_APERTURA
 $Comp
-L power:+5V #PWR?
+L power:+5V #PWR0124
 U 1 1 60E5F3D9
 P 4350 1300
-F 0 "#PWR?" H 4350 1150 50  0001 C CNN
+F 0 "#PWR0124" H 4350 1150 50  0001 C CNN
 F 1 "+5V" V 4365 1428 50  0000 L CNN
 F 2 "" H 4350 1300 50  0001 C CNN
@@
 $EndComp
 $Comp
-L power:+3.3V #PWR?
+L power:+3.3V #PWR0125
 U 1 1 60E5F3DF
 P 4350 1400
-F 0 "#PWR?" H 4350 1250 50  0001 C CNN
+F 0 "#PWR0125" H 4350 1250 50  0001 C CNN
 F 1 "+3.3V" V 4365 1528 50  0000 L CNN
 F 2 "" H 4350 1400 50  0001 C CNN
@@
 	4350 1400 4550 1400
 $Comp
-L power:GND #PWR?
+L power:GND #PWR0126
 U 1 1 60E5F3E7
 P 4350 1500
-F 0 "#PWR?" H 4350 1250 50  0001 C CNN
+F 0 "#PWR0126" H 4350 1250 50  0001 C CNN
 F 1 "GND" V 4355 1372 50  0000 R CNN
 F 2 "" H 4350 1500 50  0001 C CNN
@@
 S_APERTURA
 $Sheet
-S 4550 1050 1550 2250
+S 4550 1050 1400 2550
 U 60989480
 F0 "esp32" 50
@@
 F17 "CS" O L 4550 2900 50
 F18 "DIO0" O L 4550 3000 50
+F19 "TX_SWITCH" O L 4550 3100 50
+F20 "RX_SWITCH" O L 4550 3200 50
 $EndSheet
 Wire Wire Line
@@
 	7000 5050 7200 5050
 $Comp
-L power:+3.3V #PWR?
+L power:+3.3V #PWR0127
 U 1 1 60E895C7
 P 7000 4550
-F 0 "#PWR?" H 7000 4400 50  0001 C CNN
+F 0 "#PWR0127" H 7000 4400 50  0001 C CNN
 F 1 "+3.3V" V 7015 4678 50  0000 L CNN
 F 2 "" H 7000 4550 50  0001 C CNN
@@
 $EndComp
 $Comp
-L power:+5V #PWR?
+L power:+5V #PWR0128
 U 1 1 60E8A1FB
 P 7000 4450
-F 0 "#PWR?" H 7000 4300 50  0001 C CNN
+F 0 "#PWR0128" H 7000 4300 50  0001 C CNN
 F 1 "+5V" V 7015 4578 50  0000 L CNN
 F 2 "" H 7000 4450 50  0001 C CNN
@@
 $EndComp
 $Comp
-L power:GND #PWR?
+L power:GND #PWR0129
 U 1 1 60E8BB2F
 P 7000 4650
-F 0 "#PWR?" H 7000 4400 50  0001 C CNN
+F 0 "#PWR0129" H 7000 4400 50  0001 C CNN
 F 1 "GND" V 7005 4522 50  0000 R CNN
 F 2 "" H 7000 4650 50  0001 C CNN
@@
 F13 "SCK" B L 7200 5550 50
 F14 "CS" B L 7200 5650 50
+F15 "RX_SWITCH" I L 7200 5850 50
+F16 "TX_SWITCH" I L 7200 5750 50
 $EndSheet
 Wire Wire Line
@@
 Text Label 4350 3000 2    50   ~ 0
 DIO0
+Text Label 4350 3200 2    50   ~ 0
+RX_SWITCH
+Text Label 4350 3100 2    50   ~ 0
+TX_SWITCH
+Wire Wire Line
+	4550 3100 4350 3100
+Wire Wire Line
+	4350 3200 4550 3200
+Text Label 7000 5850 2    50   ~ 0
+RX_SWITCH
+Text Label 7000 5750 2    50   ~ 0
+TX_SWITCH
+Wire Wire Line
+	7200 5750 7000 5750
+Wire Wire Line
+	7000 5850 7200 5850
 $EndSCHEMATC

Commit message: avance2 19/07/2021
Changed lines of the file:
@@
 F17 "CS" O L 4550 2900 50
 F18 "DIO0" O L 4550 3000 50
-F19 "TX_SWITCH" O L 4550 3100 50
-F20 "RX_SWITCH" O L 4550 3200 50
-F21 "RELAY1" O L 4550 3300 50
-F22 "RELAY2" O L 4550 3400 50
-F23 "RELAY3" O L 4550 3500 50
-F24 "RELAY4" O L 4550 3600 50
+F19 "RELAY1" O L 4550 3300 50
+F20 "RELAY2" O L 4550 3400 50
+F21 "RELAY3" O L 4550 3500 50
+F22 "RELAY4" O L 4550 3600 50
 $EndSheet
 Wire Wire Line
@@
 F13 "SCK" B L 7200 5550 50
 F14 "CS" B L 7200 5650 50
-F15 "RX_SWITCH" I L 7200 5850 50
-F16 "TX_SWITCH" I L 7200 5750 50
 $EndSheet
 Wire Wire Line
@@
 Text Label 4350 3000 2    50   ~ 0
 DIO0
-Text Label 4350 3200 2    50   ~ 0
-RX_SWITCH
-Text Label 4350 3100 2    50   ~ 0
-TX_SWITCH
-Wire Wire Line
-	4550 3100 4350 3100
-Wire Wire Line
-	4350 3200 4550 3200
-Text Label 7000 5850 2    50   ~ 0
-RX_SWITCH
-Text Label 7000 5750 2    50   ~ 0
-TX_SWITCH
-Wire Wire Line
-	7200 5750 7000 5750
-Wire Wire Line
-	7000 5850 7200 5850
 Wire Wire Line
 	1150 1700 1600 1700
