File: Control de Gabinetes/Control de Gabinetes.kicad_pcb (KiCad board)
At the start: 2 copper layers, 13 parts, among them J1 Conn_01x03_MountingPin, J2 APERTURA, J3 MOVIMIENTO, J4 TEMPERATURA PRESION, J5 HUMEDAD, U1 ESP32-WROOM-32D, U2 LM1117-3.3, U3 LM1117-5.0

Commit message: AVANCE 13/07/2021
Parts:
- added AE1: Antenna, RF_Antenna:Texas_SWRA416_868MHz_915MHz, F.Cu at (244.3, 14.7)
- added C5: 10uf, Capacitor_SMD:C_0805_2012Metric, F.Cu at (250.2, -4.64)
- added C6: 0.1uf, Capacitor_SMD:C_0805_2012Metric, F.Cu at (231.8, 2.75)
- added D1: LED ROJO, LED_SMD:LED_0805_2012Metric, F.Cu at (265.4, -8.64)
- added D2: LED AMARILLO, LED_SMD:LED_0805_2012Metric, F.Cu at (265.4, -11.7)
- added J6: Conn_01x04, Connector_Molex:Molex_KK-254_AE-6410-04A_1x04_P2.54mm_Vertical, F.Cu at (238.0, -9.25)
- added Q1: PN2222A, Package_TO_SOT_SMD:SOT-23, F.Cu at (160.2, 16.3)
- added R10: 10K, Resistor_SMD:R_0805_2012Metric, F.Cu at (254.6, -4.67)
- added R11: 10K, Resistor_SMD:R_0805_2012Metric, F.Cu at (246.8, -1.66)
- added R12: 10K, Resistor_SMD:R_0805_2012Metric, F.Cu at (242.4, -3.87)
- added R13: R0, Resistor_SMD:R_0805_2012Metric, F.Cu at (193.0, -11.4)
- added R14: R0, Resistor_SMD:R_0805_2012Metric, F.Cu at (193.0, -8.48)
- added R15: 4.7K, Resistor_SMD:R_0805_2012Metric, F.Cu at (164.6, 15.5)
- added R16: 47K, Resistor_SMD:R_0805_2012Metric, F.Cu at (164.6, 18.4)
- added R2: 0, Resistor_SMD:R_0805_2012Metric, F.Cu at (269.8, -11.7)
- added R3: 0, Resistor_SMD:R_0805_2012Metric, F.Cu at (269.8, -8.77)
- added R4: 10K, Resistor_SMD:R_0805_2012Metric, F.Cu at (274.2, -11.7)
- added R5: 10K, Resistor_SMD:R_0805_2012Metric, F.Cu at (274.2, -8.77)
- added R6: 10K, Resistor_SMD:R_0805_2012Metric, F.Cu at (265.3, -0.64)
- added R7: 10K, Resistor_SMD:R_0805_2012Metric, F.Cu at (265.3, 2.31)
- added R8: 20K, Resistor_SMD:R_0805_2012Metric, F.Cu at (269.7, -0.64)
- added R9: 10K, Resistor_SMD:R_0805_2012Metric, F.Cu at (269.7, 2.31)
- added SW1: SW_Push, Button_Switch_SMD:SW_SPST_TL3342, F.Cu at (252.7, -9.67)
- added U4: RF-LORA-915-SO, RF-LORA-868-SO:XCVR_RF-LORA-868-SO, F.Cu at (245.9, 36.2)
- added U5: SIM7600SA, SIM7600SA:SIM7600SA, F.Cu at (156.2, 14.1)
- C1, C2: value 100nf -> 0.1uf
Connections:
- C3 pad 1: +5V -> Net-(C3-Pad1)
- C4 pad 1: +3V3 -> Net-(C4-Pad1)
- J2 pad 2: /sensores/S_APERTURA -> /S_APERTURA
- J3 pad 2: /sensores/S_MOVIMIENTO -> Net-(J3-Pad2)
- J4 pad 3: /sensores/SCL -> /SCL
- J4 pad 4: /sensores/SDA -> /SDA
- J5 pad 2: /sensores/S_HUMEDAD -> Net-(J5-Pad2)
- R1 pad 1: /sensores/S_APERTURA -> /S_APERTURA
- U1 pad 1: Net-(U1-Pad1) -> GND
- U1 pad 10: Net-(U1-Pad10) -> /SLEEP1
- U1 pad 11: Net-(U1-Pad11) -> /RESET_L
- U1 pad 12: Net-(U1-Pad12) -> /DIO0
- U1 pad 13: Net-(U1-Pad13) -> /S_APERTURA
- U1 pad 14: Net-(U1-Pad14) -> /S_HUMEDAD
- U1 pad 15: Net-(U1-Pad1) -> GND
- U1 pad 16: Net-(U1-Pad16) -> /S_MOVIMIENTO
- U1 pad 2: Net-(U1-Pad2) -> +3V3
- U1 pad 23: Net-(U1-Pad23) -> /PWRKEY
- U1 pad 27: Net-(U1-Pad27) -> /RX2
- U1 pad 28: Net-(U1-Pad28) -> /TX2
- U1 pad 29: Net-(U1-Pad29) -> /CS
- U1 pad 3: Net-(U1-Pad3) -> /esp32/RESET
- U1 pad 30: Net-(U1-Pad30) -> /SCK
- U1 pad 31: Net-(U1-Pad31) -> /MISO
- U1 pad 33: Net-(U1-Pad33) -> /SDA
- U1 pad 34: Net-(U1-Pad34) -> /esp32/RX
- U1 pad 35: Net-(U1-Pad35) -> /esp32/TX
- U1 pad 36: Net-(U1-Pad36) -> /SCL
- U1 pad 37: Net-(U1-Pad37) -> /MOSI
- U1 pad 38: Net-(U1-Pad1) -> GND
- U1 pad 39: Net-(U1-Pad1) -> GND
- U1 pad 8: Net-(U1-Pad8) -> /TX_SWITCH
- U1 pad 9: Net-(U1-Pad9) -> /RX_SWITCH
- U2 pad 2: +3V3 -> Net-(C4-Pad1)
- U3 pad 2: +5V -> Net-(C3-Pad1)

Commit message: avance 19/07
Parts:
- added D3: US1J, Diode_SMD:D_SMA, F.Cu at (258.0, -7.77)
- added D4: US1J, Diode_SMD:D_SMA, F.Cu at (299.3, -41.3)
- added D5: US1J, Diode_SMD:D_SMA, F.Cu at (286.1, -25.6)
- added D6: US1J, Diode_SMD:D_SMA, F.Cu at (266.0, -7.77)
- added J10: Screw_Terminal_01x02, TerminalBlock:TerminalBlock_bornier-2_P5.08mm, F.Cu at (273.8, -32.4)
- added J11: Conn_01x02_Male, Connector_PinHeader_2.54mm:PinHeader_1x02_P2.54mm_Vertical, F.Cu at (258.9, -9.52)
- added J12: Conn_01x02_Male, Connector_PinHeader_2.54mm:PinHeader_1x02_P2.54mm_Vertical, F.Cu at (263.5, -9.52)
- added J13: Conn_01x02_Male, Connector_PinHeader_2.54mm:PinHeader_1x02_P2.54mm_Vertical, F.Cu at (268.2, -9.52)
- added J7: Screw_Terminal_01x02, TerminalBlock:TerminalBlock_bornier-2_P5.08mm, F.Cu at (273.8, -14.3)
- added J8: Screw_Terminal_01x02, TerminalBlock:TerminalBlock_bornier-2_P5.08mm, F.Cu at (285.3, -32.4)
- added J9: Screw_Terminal_01x02, TerminalBlock:TerminalBlock_bornier-2_P5.08mm, F.Cu at (273.8, -23.3)
- added K1: FINDER-36.11, Relay_THT:Relay_SPDT_Finder_36.11, F.Cu at (252.2, -18.4)
- added K2: FINDER-36.11, Relay_THT:Relay_SPDT_Finder_36.11, F.Cu at (231.5, -35.2)
- added K3: FINDER-36.11, Relay_THT:Relay_SPDT_Finder_36.11, F.Cu at (252.2, -35.2)
- added K4: FINDER-36.11, Relay_THT:Relay_SPDT_Finder_36.11, F.Cu at (231.5, -18.4)
- added Q2: PN2222A, Package_TO_SOT_THT:TO-92_Inline, F.Cu at (295.6, -33.7)
- added Q3: PN2222A, Package_TO_SOT_THT:TO-92_Inline, F.Cu at (272.0, -6.50)
- added Q4: PN2222A, Package_TO_SOT_THT:TO-92_Inline, F.Cu at (284.1, -20.1)
- added Q5: PN2222A, Package_TO_SOT_THT:TO-92_Inline, F.Cu at (295.6, -27.9)
- added Q6: PN2222A, Package_TO_SOT_THT:TO-92_Inline, F.Cu at (237.7, 11.7)
- added Q7: PN2222A, Package_TO_SOT_THT:TO-92_Inline, F.Cu at (240.8, 4.65)
- added Q8: PN2222A, Package_TO_SOT_THT:TO-92_Inline, F.Cu at (231.2, 11.7)
- added R17: 500, Resistor_SMD:R_0805_2012Metric, F.Cu at (265.0, -4.02)
- added R18: 500, Resistor_SMD:R_0805_2012Metric, F.Cu at (256.2, -4.02)
- added R19: 500, Resistor_SMD:R_0805_2012Metric, F.Cu at (288.7, -15.9)
- added R20: 500, Resistor_SMD:R_0805_2012Metric, F.Cu at (283.2, -8.28)
- added R21: 2.2K, Resistor_SMD:R_0805_2012Metric, F.Cu at (278.8, -5.33)
- added R22: 2.2K, Resistor_SMD:R_0805_2012Metric, F.Cu at (290.8, -18.9)
- added R23: 2.2K, Resistor_SMD:R_0805_2012Metric, F.Cu at (284.3, -13.1)
- added R24: 2.2K, Resistor_SMD:R_0805_2012Metric, F.Cu at (295.2, -23.9)
- added R25: 10K, Resistor_SMD:R_0805_2012Metric, F.Cu at (260.6, -4.02)
- added R26: 10K, Resistor_SMD:R_0805_2012Metric, F.Cu at (278.8, -8.28)
- added R27: 10K, Resistor_SMD:R_0805_2012Metric, F.Cu at (284.3, -16.0)
- added R28: 10K, Resistor_SMD:R_0805_2012Metric, F.Cu at (290.8, -21.8)
- added R29: R, Resistor_SMD:R_0805_2012Metric, F.Cu at (274.8, -46.5)
- added R30: R, Resistor_SMD:R_0805_2012Metric, F.Cu at (274.8, -43.5)
- added R31: R, Resistor_SMD:R_0805_2012Metric, F.Cu at (279.2, -46.5)
- added R32: 10K, Resistor_SMD:R_0805_2012Metric, F.Cu at (247.5, 2.87)
- added SW2: ARRANQUE, Button_Switch_SMD:SW_SPST_TL3342, F.Cu at (234.0, 4.92)
- added U6: SFH6156-2T, SFH6156-2T:SOT254P978X405-4N, F.Cu at (289.1, -40.1)
- added U7: SFH6156-2T, SFH6156-2T:SOT254P978X405-4N, F.Cu at (247.8, -6.63)
- added U8: SFH6156-2T, SFH6156-2T:SOT254P978X405-4N, F.Cu at (235.4, -6.63)
- added U9: SFH6156-2T, SFH6156-2T:SOT254P978X405-4N, F.Cu at (276.7, -40.1)
- J6: footprint Connector_Molex:Molex_KK-254_AE-6410-04A_1x04_P2.54mm_Vertical -> Connector_Molex:Molex_KK-254_AE-6410-05A_1x05_P2.54mm_Vertical
- SW1: value SW_Push -> RESET
Connections:
- J6 pad 4: GND -> /esp32/DTR
- R10 pad 1: /esp32/RESET -> /esp32/EN
- SW1 pad 2: /esp32/RESET -> /esp32/EN
- U1 pad 17: Net-(U1-Pad17) -> /RELAY1
- U1 pad 18: Net-(U1-Pad18) -> /RELAY1
- U1 pad 24: Net-(U1-Pad24) -> /esp32/IO2
- U1 pad 25: Net-(U1-Pad25) -> /esp32/IO0
- U1 pad 3: /esp32/RESET -> /esp32/EN
- U1 pad 6: Net-(U1-Pad6) -> /RELAY1
- U1 pad 7: Net-(U1-Pad7) -> /RELAY1

Commit message: avance2 19/07/2021
Parts:
- added D7: LED, LED_SMD:LED_0805_2012Metric, F.Cu at (189.9, 96.3)
- added D8: LED, LED_SMD:LED_0805_2012Metric, F.Cu at (185.4, 96.3)
- Q2, Q3, Q4, Q5, Q6, Q7, Q8: footprint Package_TO_SOT_THT:TO-92_Inline -> Package_TO_SOT_SMD:SOT-23
- R29, R30, R31: value R -> 10K
- U1: footprint RF_Module:ESP32-WROOM-32 -> RF_Module:ESP32-WROOM-32U
- moved J10 262.4 mm to (56.6, 115.0), turned to 270 degrees
- moved J8 255.5 mm to (56.6, 81.6), turned to 90 degrees
- moved J9 250.1 mm to (56.6, 100.8), turned to 90 degrees
- moved Q5 249.5 mm to (93.0, 117.5), turned to 180 degrees
- moved D4 243.8 mm to (87.2, 79.0), turned to 270 degrees
- moved R24 240.6 mm to (100.5, 117.5), turned to 270 degrees
- moved R28 238.6 mm to (97.1, 117.5), turned to 270 degrees
- moved D5 234.3 mm to (87.2, 98.3), turned to 270 degrees
- moved U9 231.7 mm to (107.1, 117.7), turned to 270 degrees
- moved J7 230.2 mm to (56.6, 62.3), turned to 90 degrees
- moved Q4 225.2 mm to (92.4, 98.3), turned to 180 degrees
- moved Q2 223.6 mm to (92.4, 59.8), turned to 180 degrees
- moved R27 219.6 mm to (96.9, 98.3), turned to 270 degrees
- moved D6 218.4 mm to (87.2, 117.5), turned to 270 degrees
- moved K3 217.1 mm to (81.0, 98.3), turned to 180 degrees
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Connections:
- Q1 pad 3: /PWRKEY -> /comunicacion/POWERKEY
- R13 pad 2: /RX_SWITCH -> Net-(D7-Pad2)
- R14 pad 2: /TX_SWITCH -> Net-(D8-Pad2)
- R18 pad 2: /RELAY1 -> /RELAY2
- R19 pad 2: /RELAY1 -> /RELAY3
- R20 pad 2: /RELAY1 -> /RELAY4
- U1 pad 14: /S_HUMEDAD -> /S_MOVIMIENTO
- U1 pad 16: /S_MOVIMIENTO -> /S_HUMEDAD
- U1 pad 17: /RELAY1 -> Net-(U1-Pad17)
- U1 pad 18: /RELAY1 -> Net-(U1-Pad18)
- U1 pad 7: /RELAY1 -> /RELAY2
- U1 pad 8: /TX_SWITCH -> /RELAY3
- U1 pad 9: /RX_SWITCH -> /RELAY4
- U5 pad 4: /PWRKEY -> /comunicacion/POWERKEY

Commit message: avance 20/07/2021
Parts:
- removed R10, R32: 10K, Resistor_SMD:R_0805_2012Metric
- added C7: 0.1uf, Capacitor_SMD:C_0805_2012Metric, F.Cu at (168.8, 80.2)
- added C8: 0.1uf, Capacitor_SMD:C_0805_2012Metric, F.Cu at (168.8, 95.8)
- added H1: MountingHole, MountingHole:MountingHole_3.5mm, F.Cu at (109.7, 53.6)
- added H2: MountingHole, MountingHole:MountingHole_3.5mm, F.Cu at (217.3, 120.1)
- added H3: MountingHole, MountingHole:MountingHole_3.5mm, F.Cu at (109.5, 120.3)
- AE1: footprint RF_Antenna:Texas_SWRA416_868MHz_915MHz -> RF-LORA-868-SO:Texas_SWRA416_868MHz_915MHz
- J10, J7, J8, J9: footprint TerminalBlock:TerminalBlock_bornier-2_P5.08mm -> TerminalBlockjuan:TerminalBlock_bornier-2_P5.08mm
- moved AE1 51.1 mm to (213.1, 60.9)
- moved R13 45.2 mm to (194.4, 53.8)
- moved R14 45.2 mm to (189.9, 53.8)
- moved U4 45.2 mm to (191.8, 66.6)
- moved D7 45.2 mm to (194.4, 51.4)
- moved D8 45.2 mm to (189.9, 51.4)
- moved U5 33.6 mm to (193.4, 102.5)
- moved R15 32.5 mm to (192.3, 102.5)
- moved R16 32.5 mm to (189.1, 102.5)
- moved Q1 32.5 mm to (185.1, 102.5)
- moved J2 21.7 mm to (150.6, 120.8)
- moved R1 21.7 mm to (147.9, 113.6)
- moved R9 20.4 mm to (139.6, 108.9)
- moved R6 20.4 mm to (139.6, 113.6)
- moved J5 20.2 mm to (142.1, 120.8)
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Connections:
- net Net-(AE1-Pad1) renamed /comunicacion/ANT
- R21 pad 1: Net-(R21-Pad1) -> GND
- U1 pad 10: /SLEEP1 -> /S_MOVIMIENTO
- U1 pad 11: /RESET_L -> /S_HUMEDAD
- U1 pad 12: /DIO0 -> /S_APERTURA
- U1 pad 13: /S_APERTURA -> /DIO0
- U1 pad 14: /S_MOVIMIENTO -> /RESET_L
- U1 pad 16: /S_HUMEDAD -> /PWRKEY
- U1 pad 23: /PWRKEY -> /SLEEP1
Routing:
- net +5V: track 0.00 -> 356.5 mm
- net +3V3: track 0.00 -> 174.5 mm, vias 0 -> 1
- net /DIO0: track 0.00 -> 139.0 mm
- net /RESET_L: track 0.00 -> 81.5 mm, vias 0 -> 1
- net /PWRKEY: track 0.00 -> 71.5 mm
- net /CS: track 0.00 -> 60.7 mm
- net +12V: track 0.00 -> 60.5 mm, vias 0 -> 2
- net /esp32/EN: track 0.00 -> 59.9 mm, vias 0 -> 2
- net /MOSI: track 0.00 -> 59.5 mm
- net /MISO: track 0.00 -> 55.8 mm
- net /SCL: track 0.00 -> 53.0 mm, vias 0 -> 1
- net /SCK: track 0.00 -> 53.0 mm
- net /esp32/RX: track 0.00 -> 52.7 mm
- net /esp32/IO0: track 0.00 -> 50.1 mm, vias 0 -> 1
- net /actuadores/LINEA1: track 0.00 -> 50.0 mm
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- added copper zone on B.Cu, net GND
- added copper zone on F.Cu, net GND
- added copper zone on F.Cu, net Net-(C3-Pad1)
- added copper zone on F.Cu, net Net-(C4-Pad1)
Other:
- board outline added: 156 x 79 mm
- net class 5 mm added: clearance 0.5, trace_width 0.5, via_dia 0.8, via_drill 0.4
- net class Default: clearance 0.2 -> 0.5
- rule trace_clearance: 0.2 -> 0.5
- board text added: "+"
